File: client_board/client_board.brd (EAGLE design)
At the start: 65 x 56 mm, 21 parts, among them IC1 V7805-1000, J2 PJ-102AH, J3 SFH11-PBPC-D20-ST-BK

Commit message: picam360
Other:
- board text added: "Picam360"
- board text removed: "OpenBLW"
Changed lines of the file:
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@@
 <wire x1="3.6" y1="56" x2="0" y2="52.4" width="0" layer="20" curve="90"/>
 <wire x1="0" y1="52.4" x2="0" y2="3.6" width="0" layer="20"/>
-<text x="25.654" y="50.8" size="2.54" layer="21" rot="R180">OpenBLW</text>
+<text x="25.654" y="50.8" size="2.54" layer="21" rot="R180">Picam360</text>
 <text x="10.16" y="44.831" size="1.6764" layer="21">Client Board</text>
 <text x="10.16" y="42.291" size="1.4224" layer="21">Rev.0.1</text>
