File: rpcm_board/rpcm_board.brd (EAGLE design)
At the start: 72 x 56 mm, 45 parts, among them U1 SFW15R-1STE1LF, U2 SFW15R-1STE1LF, U3 DMG1012T, U5 PAM2306DYPAA

Commit message: bom
Parts:
- moved C2 3.62 mm to (23.4, 5.80)
- moved C6 3.62 mm to (23.4, 3.77)
- moved C1 3.49 mm to (18.9, 14.0)
- moved C3 3.49 mm to (23.0, 12.0)
- moved C7 3.49 mm to (23.0, 14.0)
- moved L2 3.49 mm to (28.1, 12.5)
- moved R1 3.49 mm to (18.9, 12.5)
- moved R2 3.49 mm to (26.9, 7.87)
- moved R5 3.49 mm to (30.0, 7.87)
- moved U5 3.49 mm to (23.0, 9.21)
- moved L1 3.49 mm to (17.9, 5.14)
- moved C5 3.49 mm to (17.5, 9.21)
- moved R3 3.49 mm to (18.8, 9.21)
- moved R4 3.49 mm to (16.3, 9.21)
- moved C4 3.49 mm to (28.5, 7.87)
- renumbered U$1 to U4
Connections:
- net +3V3: no longer R7.2
- net +5V: now also R7.2
Routing:
- net +5V: track 140.1 -> 45.5 mm, vias 6 -> 8
- net CAM1_IO0: track 64.3 -> 59.7 mm
- net CAM1_IO1: track 62.5 -> 58.0 mm
- net CAM0_SCL: track 42.2 -> 45.1 mm, vias 1 -> 2
- net CAM1_SCL: track 133.5 -> 131.0 mm, vias 3 -> 4
- net +1V8: track 45.8 -> 47.8 mm
- net SDX_D1: track 79.2 -> 78.2 mm
- net CAM1_SDA: track 133.9 -> 134.5 mm, vias 3 -> 4
- net GND: vias 252 -> 223
- added copper zone on layer 1, net +5V
- added copper zone on layer 16, net +5V
Other:
- board text added: "Rev.0.7"
- board text removed: "Rev.0.6"

Commit message: before hdmi
Parts:
- added JP4: (no value), openblw:1X02
- JP2: device pinhead:2X08 -> pinhead+:2X10
- R11, R12: value 100K -> 1.8K
- moved JP6 5.12 mm to (30.9, 1.50)
- moved R5 3.50 mm to (26.5, 7.87)
- moved C4 3.30 mm to (25.2, 7.87)
- moved R2 3.00 mm to (23.9, 7.87)
- moved C1 2.90 mm to (16.0, 14.0)
- moved C3 2.90 mm to (20.1, 12.0)
- moved C7 2.90 mm to (20.1, 14.0)
- moved R1 2.90 mm to (16.0, 12.5)
- moved U5 2.90 mm to (20.1, 9.21)
- moved C5 2.90 mm to (14.6, 9.21)
- moved L1 2.90 mm to (15.0, 5.14)
- moved R4 2.90 mm to (13.4, 9.21)
- moved C2 2.90 mm to (20.5, 5.80)
- moved C6 2.90 mm to (20.5, 3.77)
- moved L2 2.90 mm to (25.2, 12.5)
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Connections:
- removed net N$31: PCB1.82, R12.1
- removed net N$34: PCB1.84, R11.1
- new net GPIO44: JP2.3, PCB1.82, R12.1
- new net GPIO45: JP2.5, PCB1.84, R11.1
- net +3V3: now also JP2.17, R11.2, R12.2
- net CAM0_SCL: no longer JP2.5
- net CAM0_SDA: no longer JP2.3
- net GND: now also JP2.20; no longer R11.2, R12.2
- net GPIO42: now also JP2.18
- net GPIO43: now also JP2.19
- net USB_D_N: now also JP4.1
- net USB_D_P: now also JP4.2
Routing:
- net GPIO44: track 0.00 -> 46.4 mm, vias 0 -> 3
- net GPIO45: track 0.00 -> 45.7 mm, vias 0 -> 3
- net GPIO42: track 0.00 -> 35.3 mm
- net GPIO43: track 0.00 -> 32.7 mm
- net CAM0_SCL: track 45.1 -> 28.2 mm, vias 2 -> 1
- net +3V3: track 248.0 -> 260.9 mm
- net CAM0_SDA: track 41.4 -> 33.3 mm
- net +5V: track 45.5 -> 38.9 mm, vias 8 -> 11
- net N$31: track 4.94 -> 0.00 mm, vias 1 -> 0
- net N$34: track 4.86 -> 0.00 mm, vias 1 -> 0
- net SDX_D3: track 75.2 -> 77.9 mm
- net SDX_D2: track 77.3 -> 80.0 mm
- net SDX_D0: track 78.1 -> 80.8 mm
- net SDX_CMD: track 77.8 -> 80.5 mm
- net SDX_D1: track 78.2 -> 80.9 mm
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
Commit message: after hdmi
Parts:
- added C8: 100n, rcl:C0603
- added D2, D3, D4, D6: BAV99, diode:SOT23
- added D5: BAT54, diode:SOT23
- added HDMI: HDMI, raspi:HDMI
- added Q4: DMG1012T, transistor-fet:SC75_INFINEON
- added R10: 100k, rcl:R0603
- added R18, R19: 1k8, rcl:R0603
- moved JP3 69.0 mm to (70.5, 13.3), turned to 90 degrees
- moved U2 59.1 mm to (63.6, 38.9), turned to 90 degrees
- moved R17 53.2 mm to (62.2, 34.2), turned to 0 degrees
- moved R16 52.7 mm to (62.2, 32.6), turned to 0 degrees
- moved JP4 15.2 mm to (15.7, 6.72)
- moved JP6 14.9 mm to (16.0, 1.50)
- moved LED1 10.9 mm to (16.4, 47.0)
- moved LED2 10.9 mm to (16.4, 48.1)
- moved R15 10.9 mm to (13.5, 48.1)
- moved R6 10.9 mm to (13.5, 47.0)
- moved U3 10.9 mm to (19.7, 47.8)
- moved U4 9.40 mm to (27.7, 7.20)
- moved R9 8.83 mm to (9.86, 40.1)
- moved R8 8.81 mm to (7.29, 40.1)
- moved R7 8.81 mm to (4.72, 40.1)
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Connections:
- new net 1V8: R10.2
- new net 5V_HDMI: C8.1, D2.2, D3.2, D4.2, D5.3, D6.2, HDMI.18
- new net GPIO46: PCB1.88, Q4.2, R10.1
- new net HDMI_CEC: D4.3, HDMI.13, PCB1.171
- new net HDMI_CK_N: HDMI.12, PCB1.111
- new net HDMI_CK_P: HDMI.10, PCB1.113
- new net HDMI_D0_N: HDMI.9, PCB1.117
- new net HDMI_D0_P: HDMI.7, PCB1.119
- new net HDMI_D1_N: HDMI.6, PCB1.123
- new net HDMI_D1_P: HDMI.4, PCB1.125
- new net HDMI_D2_N: HDMI.3, PCB1.129
- new net HDMI_D2_P: HDMI.1, PCB1.131
- new net HDMI_SCL: D3.3, HDMI.15, PCB1.175, R19.1
- new net HDMI_SDA: D2.3, HDMI.16, PCB1.173, R18.1
- new net N$34: D6.3, HDMI.19, Q4.1
- net +5V: now also D5.1, R18.2, R19.2
- net GND: now also C8.2, D2.1, D3.1, D4.1, D6.1, HDMI.11, HDMI.17, HDMI.2, HDMI.5, HDMI.8, HDMI.P$1, HDMI.P$2, HDMI.P$3, HDMI.P$4, Q4.3
Routing:
- net CAM1_SDA: track 134.5 -> 76.0 mm, vias 4 -> 2
- net CAM1_SCL: track 131.0 -> 75.8 mm, vias 4 -> 2
- net 5V_HDMI: track 0.00 -> 46.6 mm, vias 0 -> 2
- net HDMI_CK_N: track 0.00 -> 44.3 mm, vias 0 -> 1
- net HDMI_CK_P: track 0.00 -> 43.9 mm, vias 0 -> 1
- net HDMI_D0_N: track 0.00 -> 41.7 mm, vias 0 -> 1
- net HDMI_D0_P: track 0.00 -> 41.3 mm, vias 0 -> 1
- net CAM1_IO0: track 59.7 -> 18.7 mm, vias 3 -> 1
- net CAM1_IO1: track 58.0 -> 18.5 mm, vias 3 -> 1
- net HDMI_D1_N: track 0.00 -> 39.2 mm, vias 0 -> 1
- net HDMI_CEC: track 0.00 -> 39.0 mm, vias 0 -> 5
- net HDMI_D1_P: track 0.00 -> 38.8 mm, vias 0 -> 1
- net HDMI_D2_N: track 0.00 -> 36.8 mm, vias 0 -> 1
- net HDMI_SCL: track 0.00 -> 36.6 mm, vias 0 -> 3
- net HDMI_D2_P: track 0.00 -> 36.3 mm, vias 0 -> 1
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Other:
- board text removed: "PWR"

Commit message: before autorouter
Parts:
- C8: device rcl:C0603 -> resistor:C0402
- Q4: device transistor-fet:SC75_INFINEON -> openblw:SOT523
- R10, R18, R19: device rcl:R0603 -> resistor:R0402
- moved LOGO1 3.55 mm to (52.1, 24.9)
- moved Q4 2.10 mm to (15.5, 23.0), turned to 90 degrees
- moved R10 0.70 mm to (17.3, 23.9), turned to 90 degrees
- moved R18 0.20 mm to (11.4, 30.9)
- moved C8 0.20 mm to (23.0, 30.9)
- moved R19 0.20 mm to (8.10, 30.9)
Connections:
- removed net 1V8: R10.2
- net +1V8: now also R10.2
- net GND: now also Q4.2; no longer Q4.3
- net GPIO46: now also Q4.3; no longer Q4.2
Routing:
- net +1V8: track 82.6 -> 97.4 mm, vias 2 -> 4
- net N$34: track 26.3 -> 28.8 mm
- net GPIO46: track 31.4 -> 32.6 mm
Other:
- board text added: "PWR"
- board text added: "Rev.0.8"
- board text removed: "CAM1"
- board text removed: "Rev.0.7"

Commit message: hdmi
Parts:
- HDMI: value HDMI -> 10029449-111RLF
Changed lines of the file:
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@@
 <attribute name="VALUE" x="13.14" y="3.545" size="1.27" layer="27"/>
 </element>
-<element name="HDMI" library="raspi" package="HDMI" value="HDMI" x="5.5" y="16.3" smashed="yes" rot="MR90">
+<element name="HDMI" library="raspi" package="HDMI" value="10029449-111RLF" x="5.5" y="16.3" smashed="yes" rot="MR90">
 <attribute name="NAME" x="12.04" y="16.54" size="1.016" layer="26" rot="MR90"/>
 </element>

Commit message: camera_unit 0.3
Parts:
- moved JP4 0.59 mm to (15.7, 7.31)
Changed lines of the file:
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@@
 <attribute name="PROD_ID" value="CONN-09505" x="70.5" y="13.3" size="1.778" layer="27" rot="R90" display="off"/>
 </element>
-<element name="JP4" library="openblw" package="1X02" value="" x="15.68" y="6.72" smashed="yes">
-<attribute name="NAME" x="13.0638" y="8.5488" size="0.6096" layer="25" ratio="10"/>
-<attribute name="VALUE" x="13.14" y="3.545" size="1.27" layer="27"/>
+<element name="JP4" library="openblw" package="1X02" value="" x="15.68" y="7.31" smashed="yes">
+<attribute name="NAME" x="13.3638" y="8.8388" size="0.6096" layer="25" ratio="10"/>
+<attribute name="VALUE" x="13.14" y="4.135" size="1.27" layer="27"/>
 </element>
 <element name="HDMI" library="raspi" package="HDMI" value="10029449-111RLF" x="5.5" y="16.3" smashed="yes" rot="MR90">
@@
 <vertex x="2" y="37.3"/>
 <vertex x="2" y="11.5"/>
-<vertex x="11.8" y="11.6"/>
+<vertex x="11.9" y="11.6"/>
 <vertex x="11.9" y="1.7"/>
 <vertex x="56.3" y="1.7"/>
@@
 <via x="38.1" y="9.7" extent="1-16" drill="0.3"/>
 <via x="19.67" y="12.34" extent="1-16" drill="0.3"/>
-<via x="14.2" y="10" extent="1-16" drill="0.3"/>
+<via x="14.3" y="10" extent="1-16" drill="0.3"/>
 <via x="24.4" y="13.9" extent="1-16" drill="0.3"/>
-<via x="12.7" y="8.1" extent="1-16" drill="0.3"/>
+<via x="12.9" y="8.4" extent="1-16" drill="0.3"/>
 <via x="38.2" y="14.9" extent="1-16" drill="0.3"/>
 <via x="23.9" y="38" extent="1-16" drill="0.3"/>
@@
 <via x="62" y="18" extent="1-16" drill="0.3"/>
 <via x="64.4" y="18" extent="1-16" drill="0.3"/>
-<via x="12.7" y="5.9" extent="1-16" drill="0.3"/>
-<via x="14.4" y="8.5" extent="1-16" drill="0.3"/>
+<via x="13.1" y="5.9" extent="1-16" drill="0.3"/>
+<via x="17.1" y="5.6" extent="1-16" drill="0.3"/>
 <via x="22.6" y="15.5" extent="1-16" drill="0.3"/>
-<via x="17.1" y="8.5" extent="1-16" drill="0.3"/>
+<via x="18.4" y="8.6" extent="1-16" drill="0.3"/>
 <via x="64.1" y="21" extent="1-16" drill="0.3"/>
 <via x="7.3" y="12.6" extent="1-16" drill="0.3"/>
@@
 <wire x1="24.2" y1="37.1" x2="24.2" y2="37.3" width="0.2" layer="1"/>
 <via x="38.3" y="12.1" extent="1-16" drill="0.3"/>
-<via x="18.9" y="9" extent="1-16" drill="0.3"/>
+<via x="18.8" y="10.1" extent="1-16" drill="0.3"/>
 <via x="37.9" y="7.1" extent="1-16" drill="0.3"/>
 <via x="31.5" y="3.6" extent="1-16" drill="0.3"/>
@@
 <via x="24.2" y="11.3" extent="1-16" drill="0.3"/>
 <via x="33.5" y="17.6" extent="1-16" drill="0.3"/>
-<via x="12.7" y="9.9" extent="1-16" drill="0.3"/>
+<via x="12.8" y="9.8" extent="1-16" drill="0.3"/>
 <via x="16.6" y="13.4" extent="1-16" drill="0.3"/>
 <via x="10.6" y="22.1" extent="1-16" drill="0.3"/>
@@
 <wire x1="14.3968" y1="31.1" x2="14.3968" y2="11.51583125" width="0.254" layer="1"/>
 <wire x1="14.3968" y1="11.51583125" x2="15.4768" y2="10.43583125" width="0.254" layer="1"/>
-<wire x1="15.4768" y1="10.43583125" x2="15.4768" y2="6.72" width="0.254" layer="1"/>
-<wire x1="15.4768" y1="6.72" x2="15.4768" y2="5.7" width="0.254" layer="1"/>
+<wire x1="15.4768" y1="10.43583125" x2="15.4768" y2="7.31" width="0.254" layer="1"/>
+<wire x1="15.4768" y1="7.31" x2="15.4768" y2="5.7" width="0.254" layer="1"/>
 <wire x1="15.4768" y1="5.7" x2="15.355" y2="5.5782" width="0.254" layer="1"/>
 <wire x1="15.355" y1="5.5782" x2="15.355" y2="4.15" width="0.254" layer="1"/>
-<wire x1="14.41" y1="6.72" x2="15.4768" y2="6.72" width="0.254" layer="1"/>
+<wire x1="14.41" y1="7.31" x2="15.4768" y2="7.31" width="0.254" layer="1"/>
 </signal>
 <signal name="USB_D_P" class="3">
@@
 <wire x1="14.8032" y1="31.1" x2="14.8032" y2="11.68416875" width="0.254" layer="1"/>
 <wire x1="14.8032" y1="11.68416875" x2="15.8832" y2="10.60416875" width="0.254" layer="1"/>
-<wire x1="15.8832" y1="10.60416875" x2="15.8832" y2="6.72" width="0.254" layer="1"/>
-<wire x1="15.8832" y1="6.72" x2="15.8832" y2="5.7" width="0.254" layer="1"/>
+<wire x1="15.8832" y1="10.60416875" x2="15.8832" y2="7.31" width="0.254" layer="1"/>
+<wire x1="15.8832" y1="7.31" x2="15.8832" y2="5.7" width="0.254" layer="1"/>
 <wire x1="15.8832" y1="5.7" x2="16.005" y2="5.5782" width="0.254" layer="1"/>
 <wire x1="16.005" y1="5.5782" x2="16.005" y2="4.15" width="0.254" layer="1"/>
-<wire x1="16.95" y1="6.72" x2="15.8832" y2="6.72" width="0.254" layer="1"/>
+<wire x1="16.95" y1="7.31" x2="15.8832" y2="7.31" width="0.254" layer="1"/>
 </signal>
 <signal name="CAM0_D0_P" class="2">
