File: rpcm_board/rpcm_board.sch (EAGLE design)
At the start: 41 parts, among them U1 SFW15R-1STE1LF, U2 SFW15R-1STE1LF, U3 DMG1012T, U5 PAM2306DYPAA

Commit message: for 2017 version
Parts:
- added JP6: USB-IDMICRO, openblw:USB-IDMICRO
- added U$1: MICROSD_SD_MODE, con-molex-microsd:MICROSD_SD_MODE
- JP2: device pinhead:PINHD-1X5 -> pinhead:PINHD-2X8
Connections:
- removed net BOTTOM_LIGHT_ENABLED: PCB1.59/GPIO17
- removed net EXT0/UART1_TX: JP1.6, PCB1.70/GPIO40
- removed net EXT1/UART1_RX: JP1.4, PCB1.72/GPIO41
- removed net LAN_RUN: PCB1.21/GPIO6
- removed net N$16: PCB1.10/NC
- removed net N$17: PCB1.12/NC
- removed net N$18: PCB1.14/NC
- removed net N$19: PCB1.16/NC
- removed net N$20: PCB1.18/NC
- removed net N$21: PCB1.20/NC
- removed net N$22: PCB1.22/NC
- removed net N$23: PCB1.24/NC
- removed net N$29: PCB1.4/NC
- removed net N$30: PCB1.6/NC
- removed net N$35: PCB1.8/NC
- removed net TOP_LIGHT_ENABLED: PCB1.57/GPIO16
- removed net UART0_RX: JP1.5, PCB1.53/GPIO15
- removed net UART0_TX: JP1.3, PCB1.51/GPIO14
- new net GPIO10: JP1.19, PCB1.33/GPIO10
- new net GPIO11: JP1.23, PCB1.35/GPIO11
- new net GPIO12: JP1.32, PCB1.45/GPIO12
- new net GPIO13: JP1.33, PCB1.47/GPIO13
- new net GPIO14: JP1.8, PCB1.51/GPIO14
- new net GPIO15: JP1.10, PCB1.53/GPIO15
- new net GPIO16: JP1.36, PCB1.57/GPIO16
- new net GPIO17: JP1.11, PCB1.59/GPIO17
- new net GPIO18: JP1.12, PCB1.63/GPIO18
- new net GPIO19: JP1.35, PCB1.65/GPIO19
- new net GPIO2: JP1.3, PCB1.9/GPIO2
- new net GPIO20: JP1.38, PCB1.69/GPIO20
- new net GPIO21: JP1.40, PCB1.71/GPIO21
- new net GPIO22: JP1.15, PCB1.75/GPIO22
- new net GPIO23: JP1.16, PCB1.77/GPIO23
- new net GPIO24: JP1.18, PCB1.81/GPIO24
- new net GPIO25: JP1.22, PCB1.83/GPIO25
- new net GPIO26: JP1.37, PCB1.87/GPIO26
- new net GPIO27: JP1.13, PCB1.89/GPIO27
- new net GPIO3: JP1.5, PCB1.11/GPIO3
- new net GPIO34: JP2.7, PCB1.52/GPIO34
- new net GPIO35: JP2.11, PCB1.54/GPIO35
- new net GPIO36: JP2.12, PCB1.58/GPIO36
- new net GPIO37: JP2.13, PCB1.60/GPIO37
- new net GPIO38: JP2.16, PCB1.64/GPIO38
- new net GPIO39: JP2.15, PCB1.66/GPIO39
- new net GPIO4: JP1.7, PCB1.15/GPIO4
- new net GPIO40: JP2.8, PCB1.70/GPIO40
- new net GPIO41: JP2.10, PCB1.72/GPIO41
- new net GPIO42: PCB1.76/GPIO42
- new net GPIO43: PCB1.78/GPIO43
- new net GPIO5: JP1.29, PCB1.17/GPIO5
- new net GPIO6: JP1.31, PCB1.21/GPIO6
- new net GPIO7: JP1.26, PCB1.23/GPIO7
- new net GPIO8: JP1.24, PCB1.27/GPIO8
- new net GPIO9: JP1.21, PCB1.29/GPIO9
- new net SDX_CLK: PCB1.10/NC, U$1.CLK
- new net SDX_CMD: PCB1.12/NC, U$1.CMD
- new net SDX_D0: PCB1.16/NC, U$1.DATA0
- new net SDX_D1: PCB1.18/NC, U$1.DATA1
- new net SDX_D2: PCB1.22/NC, U$1.DATA2
- new net SDX_D3: PCB1.24/NC, U$1.CD/DATA3
- net +1V8: no longer JP2.1
- net +3V3: now also JP1.1, JP1.17, JP2.1, PCB1.4/NC, PCB1.6/NC, U$1.VDD
- net +5V: now also JP1.4, JP2.4, JP6.VBUS; no longer JP1.1
- net CAM0_SCL: now also JP2.5
- net CAM0_SDA: now also JP2.3
- net CAM1_IO0: now also PCB1.48/GPIO33; no longer PCB1.11/GPIO3
- net CAM1_IO1: now also PCB1.46/GPIO32; no longer PCB1.9/GPIO2
- net CAM1_SCL: now also JP1.28
- net CAM1_SDA: now also JP1.27
- net GND: now also JP1.20, JP1.25, JP1.30, JP1.34, JP1.39, JP1.6, JP1.9, JP2.14, JP2.6, JP2.9, JP6.GND, PCB1.14/NC, PCB1.20/NC, PCB1.8/NC, U$1.VSS; no longer JP1.13, JP1.7, JP1.8, JP2.5
- net USB_D_N: now also JP6.D-; no longer JP2.4
- net USB_D_P: now also JP6.D+; no longer JP2.3
Other:
- note added: "UART"
- moved on the sheet: JP1, R13, R14, R16, R17

Commit message: for 2017 first version
Parts:
- U$1: value MICROSD_SD_MODE -> MICROSD_SD_MODEMOLEX; device con-molex-microsd:MICROSD_SD_MODE -> openblw:MICROSD_SD_MODEMOLEX
Changed lines of the file:
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@@
 <part name="P+1" library="supply1" deviceset="+5V" device=""/>
 <part name="JP2" library="pinhead" deviceset="PINHD-2X8" device=""/>
-<part name="U$1" library="con-molex-microsd" deviceset="MICROSD_SD_MODE" device=""/>
+<part name="U$1" library="openblw" deviceset="MICROSD_SD_MODE" device="MOLEX"/>
 <part name="GND8" library="supply" deviceset="GND" device=""/>
 <part name="V1" library="supply" deviceset="+3V3" device=""/>

Commit message: pwr
Parts:
- added JP3: USB-IDMICRO, openblw:USB-IDMICRO
Connections:
- net +5V: now also JP3.VBUS
- net GND: now also JP3.GND
Changed lines of the file:
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@@
 <part name="GND8" library="supply" deviceset="GND" device=""/>
 <part name="V1" library="supply" deviceset="+3V3" device=""/>
+<part name="JP3" library="openblw" deviceset="USB-ID" device="MICRO"/>
+<part name="P+2" library="supply1" deviceset="+5V" device=""/>
+<part name="GND11" library="supply1" deviceset="GND" device=""/>
 </parts>
 <sheets>
@@
 <instance part="GND8" gate="1" x="309.88" y="38.1"/>
 <instance part="V1" gate="G$1" x="309.88" y="86.36"/>
+<instance part="JP3" gate="G$1" x="203.2" y="119.38" rot="R270"/>
+<instance part="P+2" gate="1" x="205.74" y="152.4"/>
+<instance part="GND11" gate="1" x="203.2" y="139.7" rot="R180"/>
 </instances>
 <busses>
@@
 <pinref part="P+1" gate="1" pin="+5V"/>
 <wire x1="175.26" y1="124.46" x2="190.5" y2="124.46" width="0.1524" layer="91"/>
+</segment>
+<segment>
+<pinref part="JP3" gate="G$1" pin="VBUS"/>
+<pinref part="P+2" gate="1" pin="+5V"/>
+<wire x1="205.74" y1="121.92" x2="205.74" y2="149.86" width="0.1524" layer="91"/>
 </segment>
 </net>
@@
 <wire x1="309.88" y1="60.96" x2="309.88" y2="40.64" width="0.1524" layer="91"/>
 </segment>
+<segment>
+<pinref part="JP3" gate="G$1" pin="GND"/>
+<pinref part="GND11" gate="1" pin="GND"/>
+<wire x1="203.2" y1="121.92" x2="203.2" y2="137.16" width="0.1524" layer="91"/>
+</segment>
 </net>

Commit message: bom
Parts:
- renumbered U$1 to U4
Connections:
- net +3V3: no longer R7.2
- net +5V: now also R7.2
Changed lines of the file:
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@@
 <part name="PORT14" library="dports" deviceset="NC" device=""/>
 <part name="PORT15" library="dports" deviceset="NC" device=""/>
-<part name="V12" library="supply" deviceset="+3V3" device=""/>
 <part name="V13" library="supply" deviceset="+3V3" device=""/>
 <part name="V15" library="supply" deviceset="+1V8" device=""/>
@@
 <part name="P+1" library="supply1" deviceset="+5V" device=""/>
 <part name="JP2" library="pinhead" deviceset="PINHD-2X8" device=""/>
-<part name="U$1" library="openblw" deviceset="MICROSD_SD_MODE" device="MOLEX"/>
+<part name="U4" library="openblw" deviceset="MICROSD_SD_MODE" device="MOLEX"/>
 <part name="GND8" library="supply" deviceset="GND" device=""/>
 <part name="V1" library="supply" deviceset="+3V3" device=""/>
@@
 <part name="P+2" library="supply1" deviceset="+5V" device=""/>
 <part name="GND11" library="supply1" deviceset="GND" device=""/>
+<part name="V6" library="supply" deviceset="+5V" device=""/>
 </parts>
 <sheets>
@@
 <instance part="GND15" gate="1" x="83.82" y="149.86" rot="R180"/>
 <instance part="V10" gate="1" x="78.74" y="149.86"/>
-<instance part="V12" gate="G$1" x="350.52" y="241.3" rot="R90"/>
 <instance part="V13" gate="G$1" x="350.52" y="220.98" rot="R90"/>
 <instance part="V15" gate="G$1" x="350.52" y="200.66" rot="R90"/>
@@
 <instance part="P+1" gate="1" x="193.04" y="124.46" rot="R270"/>
 <instance part="JP2" gate="A" x="53.34" y="127" rot="R90"/>
-<instance part="U$1" gate="G$1" x="289.56" y="60.96"/>
+<instance part="U4" gate="G$1" x="289.56" y="60.96"/>
 <instance part="GND8" gate="1" x="309.88" y="38.1"/>
 <instance part="V1" gate="G$1" x="309.88" y="86.36"/>
@@
 <instance part="P+2" gate="1" x="205.74" y="152.4"/>
 <instance part="GND11" gate="1" x="203.2" y="139.7" rot="R180"/>
+<instance part="V6" gate="1" x="350.52" y="241.3" rot="R90"/>
 </instances>
 <busses>
@@
 <pinref part="P+2" gate="1" pin="+5V"/>
 <wire x1="205.74" y1="121.92" x2="205.74" y2="149.86" width="0.1524" layer="91"/>
+</segment>
+<segment>
+<pinref part="R7" gate="G$1" pin="2"/>
+<pinref part="V6" gate="1" pin="+5V"/>
+<wire x1="355.6" y1="241.3" x2="353.06" y2="241.3" width="0.1524" layer="91"/>
 </segment>
 </net>
@@
 </segment>
 <segment>
-<pinref part="U$1" gate="G$1" pin="VSS"/>
+<pinref part="U4" gate="G$1" pin="VSS"/>
 <pinref part="GND8" gate="1" pin="GND"/>
 <wire x1="302.26" y1="60.96" x2="309.88" y2="60.96" width="0.1524" layer="91"/>
@@
 </segment>
 <segment>
-<pinref part="V12" gate="G$1" pin="+3V3"/>
-<pinref part="R7" gate="G$1" pin="2"/>
-<wire x1="353.06" y1="241.3" x2="355.6" y2="241.3" width="0.1524" layer="91"/>
-</segment>
-<segment>
+<pinref part="R8" gate="G$1" pin="2"/>
 <pinref part="V13" gate="G$1" pin="+3V3"/>
-<pinref part="R8" gate="G$1" pin="2"/>
 <wire x1="353.06" y1="220.98" x2="355.6" y2="220.98" width="0.1524" layer="91"/>
 </segment>
@@
 </segment>
 <segment>
-<pinref part="U$1" gate="G$1" pin="VDD"/>
+<pinref part="U4" gate="G$1" pin="VDD"/>
 <pinref part="V1" gate="G$1" pin="+3V3"/>
 <wire x1="302.26" y1="66.04" x2="309.88" y2="66.04" width="0.1524" layer="91"/>
@@
 <net name="SDX_D2" class="0">
 <segment>
-<pinref part="U$1" gate="G$1" pin="DATA2"/>
+<pinref part="U4" gate="G$1" pin="DATA2"/>
 <wire x1="302.26" y1="73.66" x2="322.58" y2="73.66" width="0.1524" layer="91"/>
 <label x="322.58" y="73.66" size="1.778" layer="95" xref="yes"/>
@@
 <net name="SDX_D3" class="0">
 <segment>
-<pinref part="U$1" gate="G$1" pin="CD/DATA3"/>
+<pinref part="U4" gate="G$1" pin="CD/DATA3"/>
 <wire x1="302.26" y1="71.12" x2="322.58" y2="71.12" width="0.1524" layer="91"/>
 <label x="322.58" y="71.12" size="1.778" layer="95" xref="yes"/>
@@
 <net name="SDX_CMD" class="0">
 <segment>
-<pinref part="U$1" gate="G$1" pin="CMD"/>
+<pinref part="U4" gate="G$1" pin="CMD"/>
 <wire x1="302.26" y1="68.58" x2="322.58" y2="68.58" width="0.1524" layer="91"/>
 <label x="322.58" y="68.58" size="1.778" layer="95" xref="yes"/>
@@
 <net name="SDX_CLK" class="0">
 <segment>
-<pinref part="U$1" gate="G$1" pin="CLK"/>
+<pinref part="U4" gate="G$1" pin="CLK"/>
 <wire x1="302.26" y1="63.5" x2="322.58" y2="63.5" width="0.1524" layer="91"/>
 <label x="322.58" y="63.5" size="1.778" layer="95" xref="yes"/>
@@
 <net name="SDX_D0" class="0">
 <segment>
-<pinref part="U$1" gate="G$1" pin="DATA0"/>
+<pinref part="U4" gate="G$1" pin="DATA0"/>
 <wire x1="302.26" y1="58.42" x2="322.58" y2="58.42" width="0.1524" layer="91"/>
 <label x="322.58" y="58.42" size="1.778" layer="95" xref="yes"/>
@@
 <net name="SDX_D1" class="0">
 <segment>
-<pinref part="U$1" gate="G$1" pin="DATA1"/>
+<pinref part="U4" gate="G$1" pin="DATA1"/>
 <wire x1="302.26" y1="55.88" x2="322.58" y2="55.88" width="0.1524" layer="91"/>
 <label x="322.58" y="55.88" size="1.778" layer="95" xref="yes"/>

Commit message: before hdmi
Parts:
- added JP4: (no value), openblw:PINHD-1X2
- JP2: device pinhead:PINHD-2X8 -> pinhead+:PINHD-2X10
- R11, R12: value 100K -> 1.8K
Connections:
- removed net N$31: PCB1.82/GPIO44, R12.1
- removed net N$34: PCB1.84/GPIO45, R11.1
- new net GPIO44: JP2.3, PCB1.82/GPIO44, R12.1
- new net GPIO45: JP2.5, PCB1.84/GPIO45, R11.1
- net +3V3: now also JP2.17, R11.2, R12.2
- net CAM0_SCL: no longer JP2.5
- net CAM0_SDA: no longer JP2.3
- net GND: now also JP2.20; no longer R11.2, R12.2
- net GPIO42: now also JP2.18
- net GPIO43: now also JP2.19
- net USB_D_N: now also JP4.1
- net USB_D_P: now also JP4.2
Other:
- moved on the sheet: R11, R12

Commit message: after hdmi
Parts:
- added C8: 100n, rcl:C-EUC0603
- added D2, D3, D4, D6: BAV99, diode:BAV199
- added D5: BAT54, diode:BAT54
- added HDMI: HDMI, raspi:HDMI
- added Q4: DMG1012T, transistor-fet:BSA223SP
- added R10: 100k, rcl:R-EU_R0603
- added R18, R19: 1k8, rcl:R-EU_R0603
Connections:
- new net 1V8: R10.2
- new net 5V_HDMI: C8.1, D2.C, D3.C, D4.C, D5.C, D6.C, HDMI.+5V
- new net GPIO46: PCB1.88/GPIO46_1V8, Q4.D, R10.1
- new net HDMI_CEC: D4.AC, HDMI.CEC_DAT, PCB1.171/HDMI_CEC
- new net HDMI_CK_N: HDMI.CLK_N, PCB1.111/HDMI_CK_N*
- new net HDMI_CK_P: HDMI.CLK_P, PCB1.113/HDMI_CK_P*
- new net HDMI_D0_N: HDMI.TX0_N, PCB1.117/HDMI_D0_N*
- new net HDMI_D0_P: HDMI.TX0_P, PCB1.119/HDMI_D0_P*
- new net HDMI_D1_N: HDMI.TX1_N, PCB1.123/HDMI_D1_N*
- new net HDMI_D1_P: HDMI.TX1_P, PCB1.125/HDMI_D1_P*
- new net HDMI_D2_N: HDMI.TX2_N, PCB1.129/HDMI_D2_N*
- new net HDMI_D2_P: HDMI.TX2_P, PCB1.131/HDMI_D2_P*
- new net HDMI_SCL: D3.AC, HDMI.SCL, PCB1.175/HDMI_SCL, R19.1
- new net HDMI_SDA: D2.AC, HDMI.SDA, PCB1.173/HDMI_SDA, R18.1
- new net N$34: D6.AC, HDMI.HPD, Q4.G
- net +5V: now also D5.A, R18.2, R19.2
- net GND: now also C8.2, D2.A, D3.A, D4.A, D6.A, HDMI.GND@1, HDMI.GND@2, HDMI.GND@3, HDMI.GND@4, HDMI.GND@5, HDMI.GND@6, HDMI.GND@7, HDMI.GND@8, HDMI.GND@9, Q4.S

Commit message: before autorouter
Parts:
- C8: device rcl:C-EUC0603 -> resistor:C-EUC0402
- Q4: device transistor-fet:BSA223SP -> openblw:DMG1012T
- R10, R18, R19: device rcl:R-EU_R0603 -> resistor:R-EU_R0402
Connections:
- removed net 1V8: R10.2
- net +1V8: now also R10.2
Other:
- moved on the sheet: R10
Changed lines of the file:
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@@
 <part name="D4" library="diode" deviceset="BAV199" device="" value="BAV99"/>
 <part name="D5" library="diode" deviceset="BAT54" device=""/>
-<part name="C8" library="rcl" deviceset="C-EU" device="C0603" value="100n"/>
+<part name="C8" library="resistor" deviceset="C-EU" device="C0402" value="100n"/>
 <part name="GND27" library="supply1" deviceset="GND" device=""/>
 <part name="P+9" library="supply1" deviceset="+5V" device=""/>
 <part name="GND12" library="supply1" deviceset="GND" device=""/>
 <part name="D6" library="diode" deviceset="BAV199" device="" value="BAV99"/>
-<part name="R10" library="rcl" deviceset="R-EU_" device="R0603" value="100k"/>
-<part name="Q4" library="transistor-fet" deviceset="BSA223SP" device="" value="DMG1012T"/>
+<part name="R10" library="resistor" deviceset="R-EU_" device="R0402" value="100k"/>
+<part name="Q4" library="openblw" deviceset="DMG1012T" device="" value="DMG1012T"/>
 <part name="GND14" library="supply1" deviceset="GND" device=""/>
 <part name="GND30" library="supply1" deviceset="GND" device=""/>
-<part name="R18" library="rcl" deviceset="R-EU_" device="R0603" value="1k8"/>
-<part name="R19" library="rcl" deviceset="R-EU_" device="R0603" value="1k8"/>
+<part name="R18" library="resistor" deviceset="R-EU_" device="R0402" value="1k8"/>
+<part name="R19" library="resistor" deviceset="R-EU_" device="R0402" value="1k8"/>
 <part name="P+10" library="supply1" deviceset="+5V" device=""/>
 <part name="P+11" library="supply1" deviceset="+5V" device=""/>
@@
 <instance part="GND12" gate="1" x="157.48" y="40.64"/>
 <instance part="D6" gate="G$1" x="182.88" y="27.94" rot="R270"/>
-<instance part="R10" gate="G$1" x="205.74" y="33.02" rot="R90"/>
-<instance part="Q4" gate="G$1" x="203.2" y="17.78" rot="MR180"/>
-<instance part="GND14" gate="1" x="205.74" y="7.62"/>
+<instance part="R10" gate="G$1" x="238.76" y="17.78"/>
+<instance part="Q4" gate="G$1" x="205.74" y="17.78" rot="MR180"/>
+<instance part="GND14" gate="1" x="187.96" y="7.62"/>
 <instance part="GND30" gate="1" x="182.88" y="20.32"/>
 <instance part="R18" gate="G$1" x="154.94" y="86.36" rot="R90"/>
@@
 <pinref part="Q4" gate="G$1" pin="S"/>
 <pinref part="GND14" gate="1" pin="GND"/>
-<wire x1="205.74" y1="10.16" x2="205.74" y2="12.7" width="0.1524" layer="91"/>
+<wire x1="187.96" y1="10.16" x2="187.96" y2="17.78" width="0.1524" layer="91"/>
 </segment>
 <segment>
@@
 <wire x1="353.06" y1="200.66" x2="355.6" y2="200.66" width="0.1524" layer="91"/>
 </segment>
+<segment>
+<pinref part="R10" gate="G$1" pin="2"/>
+<wire x1="243.84" y1="17.78" x2="246.38" y2="17.78" width="0.1524" layer="91"/>
+<label x="246.38" y="17.78" size="1.778" layer="95" xref="yes"/>
+</segment>
 </net>
 <net name="N$2" class="0">
@@
 <wire x1="66.04" y1="132.08" x2="66.04" y2="147.32" width="0.1524" layer="91"/>
 <label x="66.04" y="147.32" size="1.778" layer="95" rot="R90" xref="yes"/>
-</segment>
-</net>
-<net name="1V8" class="0">
-<segment>
-<pinref part="R10" gate="G$1" pin="2"/>
-<wire x1="205.74" y1="38.1" x2="205.74" y2="40.64" width="0.1524" layer="91"/>
-<label x="205.74" y="40.64" size="1.778" layer="95" rot="R90" xref="yes"/>
 </segment>
 </net>
@@
 <wire x1="190.5" y1="66.04" x2="187.96" y2="66.04" width="0.1524" layer="91"/>
 <pinref part="Q4" gate="G$1" pin="G"/>
-<wire x1="200.66" y1="15.24" x2="187.96" y2="15.24" width="0.1524" layer="91"/>
-<wire x1="187.96" y1="15.24" x2="187.96" y2="27.94" width="0.1524" layer="91"/>
+<wire x1="187.96" y1="22.86" x2="187.96" y2="27.94" width="0.1524" layer="91"/>
 <pinref part="D6" gate="G$1" pin="AC"/>
 <wire x1="187.96" y1="27.94" x2="185.42" y2="27.94" width="0.1524" layer="91"/>
@@
 <pinref part="R10" gate="G$1" pin="1"/>
 <pinref part="Q4" gate="G$1" pin="D"/>
-<wire x1="205.74" y1="27.94" x2="205.74" y2="22.86" width="0.1524" layer="91"/>
-<label x="205.74" y="25.4" size="1.778" layer="95" xref="yes"/>
-</segment>
-</net>
+<wire x1="233.68" y1="17.78" x2="226.06" y2="17.78" width="0.1524" layer="91"/>
+<label x="226.06" y="20.32" size="1.778" layer="95" rot="R90" xref="yes"/>
+<wire x1="226.06" y1="17.78" x2="223.52" y2="17.78" width="0.1524" layer="91"/>
+<wire x1="226.06" y1="17.78" x2="226.06" y2="20.32" width="0.1524" layer="91"/>
+<junction x="226.06" y="17.78"/>
+</segment>
+</net>

Commit message: hdmi
Parts:
- HDMI: value HDMI -> 10029449-111RLF
Changed lines of the file:
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@@
 <part name="V9" library="supply" deviceset="+3V3" device=""/>
 <part name="JP4" library="openblw" deviceset="PINHD-1X2" device=""/>
-<part name="HDMI" library="raspi" deviceset="HDMI" device=""/>
+<part name="HDMI" library="raspi" deviceset="HDMI" device="" value="10029449-111RLF"/>
 <part name="GND26" library="supply1" deviceset="GND" device=""/>
 <part name="D2" library="diode" deviceset="BAV199" device="" value="BAV99"/>
