File: rpcm_board/rpcm_board.sch (EAGLE design)
At the start: 56 parts, among them Q4 DMG1012T, U1 SFW15R-1STE1LF, U2 SFW15R-1STE1LF, U3 DMG1012T, U4 MICROSD_SD_MODEMOLEX, U5 PAM2306DYPAA

Commit message: interface board 0.7 rpcm board 0.10
Parts:
- removed JP4: (no value), openblw:PINHD-1X2
- added C11: 4.7n, resistor:C-EUC0402
- added R20: 1M, resistor:R-EU_R0402
Connections:
- new net USB2_SHELL: C11.1, JP6.SHELL, R20.1
- net GND: now also C11.2, R20.2
- net USB_D_N: no longer JP4.1
- net USB_D_P: no longer JP4.2
Changed lines of the file:
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@@
 <?xml version="1.0" encoding="utf-8"?>
 <!DOCTYPE eagle SYSTEM "eagle.dtd">
-<eagle version="7.5.0">
+<eagle version="8.1.1">
 <drawing>
 <settings>
@@
 <part name="V6" library="supply" deviceset="+5V" device=""/>
 <part name="V9" library="supply" deviceset="+3V3" device=""/>
-<part name="JP4" library="openblw" deviceset="PINHD-1X2" device=""/>
 <part name="HDMI" library="raspi" deviceset="HDMI" device="" value="10029449-111RLF"/>
 <part name="GND26" library="supply1" deviceset="GND" device=""/>
@@
 <part name="P+10" library="supply1" deviceset="+5V" device=""/>
 <part name="P+11" library="supply1" deviceset="+5V" device=""/>
+<part name="R20" library="resistor" deviceset="R-EU_" device="R0402" value="1M"/>
+<part name="C11" library="resistor" deviceset="C-EU" device="C0402" value="4.7n"/>
 </parts>
 <sheets>
@@
 <instance part="V7" gate="G$1" x="78.74" y="106.68" rot="R180"/>
 <instance part="JP6" gate="G$1" x="172.72" y="119.38" rot="R270"/>
-<instance part="GND10" gate="1" x="157.48" y="119.38"/>
+<instance part="GND10" gate="1" x="142.24" y="119.38"/>
 <instance part="P+1" gate="1" x="193.04" y="124.46" rot="R270"/>
 <instance part="JP2" gate="A" x="55.88" y="127" rot="R90"/>
@@
 <instance part="GND11" gate="1" x="203.2" y="139.7" rot="R180"/>
 <instance part="V6" gate="1" x="350.52" y="241.3" rot="R90"/>
-<instance part="JP4" gate="G$1" x="187.96" y="147.32" rot="R90"/>
 <instance part="HDMI" gate="G$1" x="208.28" y="78.74"/>
 <instance part="GND26" gate="1" x="228.6" y="99.06" rot="R180"/>
@@
 <instance part="P+10" gate="1" x="154.94" y="99.06"/>
 <instance part="P+11" gate="1" x="160.02" y="93.98"/>
+<instance part="R20" gate="G$1" x="152.4" y="116.84" rot="R90"/>
+<instance part="C11" gate="G$1" x="157.48" y="114.3" rot="R180"/>
 </instances>
 <busses>
@@
 <wire x1="172.72" y1="121.92" x2="172.72" y2="124.46" width="0.1524" layer="91"/>
 <pinref part="GND10" gate="1" pin="GND"/>
-<wire x1="172.72" y1="124.46" x2="157.48" y2="124.46" width="0.1524" layer="91"/>
-<wire x1="157.48" y1="124.46" x2="157.48" y2="121.92" width="0.1524" layer="91"/>
+<wire x1="172.72" y1="124.46" x2="152.4" y2="124.46" width="0.1524" layer="91"/>
+<wire x1="152.4" y1="124.46" x2="142.24" y2="124.46" width="0.1524" layer="91"/>
+<wire x1="142.24" y1="124.46" x2="142.24" y2="121.92" width="0.1524" layer="91"/>
+<pinref part="C11" gate="G$1" pin="2"/>
+<wire x1="157.48" y1="119.38" x2="157.48" y2="121.92" width="0.1524" layer="91"/>
+<pinref part="R20" gate="G$1" pin="2"/>
+<wire x1="157.48" y1="121.92" x2="152.4" y2="121.92" width="0.1524" layer="91"/>
+<wire x1="152.4" y1="121.92" x2="152.4" y2="124.46" width="0.1524" layer="91"/>
+<junction x="152.4" y="121.92"/>
+<junction x="152.4" y="124.46"/>
 </segment>
 <segment>
@@
 <pinref part="JP6" gate="G$1" pin="D-"/>
 <label x="177.8" y="149.86" size="1.778" layer="95" rot="MR90" xref="yes"/>
-<wire x1="177.8" y1="121.92" x2="177.8" y2="137.16" width="0.1524" layer="91"/>
-<wire x1="177.8" y1="137.16" x2="177.8" y2="149.86" width="0.1524" layer="91"/>
-<wire x1="177.8" y1="137.16" x2="185.42" y2="137.16" width="0.1524" layer="91"/>
-<junction x="177.8" y="137.16"/>
-<pinref part="JP4" gate="G$1" pin="1"/>
-<wire x1="185.42" y1="137.16" x2="185.42" y2="144.78" width="0.1524" layer="91"/>
+<wire x1="177.8" y1="121.92" x2="177.8" y2="149.86" width="0.1524" layer="91"/>
 </segment>
 </net>
@@
 <pinref part="JP6" gate="G$1" pin="D+"/>
 <label x="180.34" y="149.86" size="1.778" layer="95" rot="MR90" xref="yes"/>
-<wire x1="180.34" y1="121.92" x2="180.34" y2="134.62" width="0.1524" layer="91"/>
-<wire x1="180.34" y1="134.62" x2="180.34" y2="149.86" width="0.1524" layer="91"/>
-<wire x1="180.34" y1="134.62" x2="187.96" y2="134.62" width="0.1524" layer="91"/>
-<junction x="180.34" y="134.62"/>
-<wire x1="187.96" y1="134.62" x2="187.96" y2="144.78" width="0.1524" layer="91"/>
-<pinref part="JP4" gate="G$1" pin="2"/>
+<wire x1="180.34" y1="121.92" x2="180.34" y2="149.86" width="0.1524" layer="91"/>
 </segment>
 </net>
@@
 </segment>
 </net>
+<net name="USB2_SHELL" class="1">
+<segment>
+<pinref part="R20" gate="G$1" pin="1"/>
+<pinref part="C11" gate="G$1" pin="1"/>
+<wire x1="152.4" y1="109.22" x2="152.4" y2="111.76" width="0.1524" layer="91"/>
+<wire x1="152.4" y1="109.22" x2="157.48" y2="109.22" width="0.1524" layer="91"/>
+<wire x1="157.48" y1="109.22" x2="157.48" y2="111.76" width="0.1524" layer="91"/>
+<junction x="152.4" y="109.22"/>
+<pinref part="JP6" gate="G$1" pin="SHELL"/>
+<wire x1="170.18" y1="116.84" x2="162.56" y2="116.84" width="0.1524" layer="91"/>
+<wire x1="162.56" y1="116.84" x2="162.56" y2="104.14" width="0.1524" layer="91"/>
+<wire x1="162.56" y1="104.14" x2="152.4" y2="104.14" width="0.1524" layer="91"/>
+<wire x1="152.4" y1="104.14" x2="152.4" y2="109.22" width="0.1524" layer="91"/>
+</segment>
+</net>

Commit message: tune value
Parts:
- R10: value 100k -> 100K
- R18, R19: value 1k8 -> 1.8K
Changed lines of the file:
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@@
 <?xml version="1.0" encoding="utf-8"?>
 <!DOCTYPE eagle SYSTEM "eagle.dtd">
-<eagle version="8.1.1">
+<eagle version="8.4.2">
 <drawing>
 <settings>
 <setting alwaysvectorfont="no"/>
+<setting keepoldvectorfont="yes"/>
 <setting verticaltext="up"/>
 </settings>
@@
 <part name="GND12" library="supply1" deviceset="GND" device=""/>
 <part name="D6" library="diode" deviceset="BAV199" device="" value="BAV99"/>
-<part name="R10" library="resistor" deviceset="R-EU_" device="R0402" value="100k"/>
+<part name="R10" library="resistor" deviceset="R-EU_" device="R0402" value="100K"/>
 <part name="Q4" library="openblw" deviceset="DMG1012T" device="" value="DMG1012T"/>
 <part name="GND14" library="supply1" deviceset="GND" device=""/>
 <part name="GND30" library="supply1" deviceset="GND" device=""/>
-<part name="R18" library="resistor" deviceset="R-EU_" device="R0402" value="1k8"/>
-<part name="R19" library="resistor" deviceset="R-EU_" device="R0402" value="1k8"/>
+<part name="R18" library="resistor" deviceset="R-EU_" device="R0402" value="1.8K"/>
+<part name="R19" library="resistor" deviceset="R-EU_" device="R0402" value="1.8K"/>
 <part name="P+10" library="supply1" deviceset="+5V" device=""/>
 <part name="P+11" library="supply1" deviceset="+5V" device=""/>
