File: interface_board/interface_board.sch (EAGLE design)
At the start: 87 parts, among them IC1 V7805-1000, IC6 LAN9512-JZX, K2 61400826021, Q1 IRLML6346TRPBF, Q6 CTS_32X25_SMD, U1 AL5812MP-13, U2 MPU-9250

Commit message: bom
Parts:
- C3: device SparkFun-Capacitors:CAP0603-CAP -> resistor:C-EUC0402
- C42: device resistor:C-EUC0603 -> resistor:C-EUC0402
- JP1: value M20-9990446 -> SSQ-108-03-G-D
- JP2, JP3: value M20-9980346 -> M20-9980345
- JP4: value (none) -> M20-9980345
- JP6: value USB-IDMICRO -> 10118192-0001LF
- Q6: value CTS_32X25_SMD -> FA-238 25.0000MB
- R1: value 4.99K -> 4.99k
- R18, R3: value 1K -> 1k
- R2: value 100K -> 100k
Changed lines of the file:
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@@
 <part name="LED1" library="openblw" deviceset="LTW-5630AZL" device="" value="LTW-5630AZL50"/>
 <part name="LED2" library="openblw" deviceset="LTW-5630AZL" device="" value="LTW-5630AZL50"/>
-<part name="R1" library="resistor" deviceset="R-EU_" device="R0402" value="4.99K"/>
+<part name="R1" library="resistor" deviceset="R-EU_" device="R0402" value="4.99k"/>
 <part name="C1" library="resistor" deviceset="C-EU" device="C0402" value="100n"/>
 <part name="GND1" library="supply" deviceset="GND" device=""/>
 <part name="GND2" library="supply" deviceset="GND" device=""/>
 <part name="GND3" library="supply" deviceset="GND" device=""/>
-<part name="R2" library="resistor" deviceset="R-EU_" device="R0402" value="100K"/>
-<part name="R3" library="resistor" deviceset="R-EU_" device="R0402" value="1K"/>
+<part name="R2" library="resistor" deviceset="R-EU_" device="R0402" value="100k"/>
+<part name="R3" library="resistor" deviceset="R-EU_" device="R0402" value="1k"/>
 <part name="GND5" library="supply" deviceset="GND" device=""/>
 <part name="GND7" library="supply" deviceset="GND" device=""/>
@@
 <part name="H3" library="holes" deviceset="MOUNT-PAD-ROUND" device="2.8"/>
 <part name="H4" library="holes" deviceset="MOUNT-PAD-ROUND" device="2.8"/>
-<part name="JP1" library="pinhead" deviceset="PINHD-2X8" device="" value="M20-9990446"/>
+<part name="JP1" library="pinhead" deviceset="PINHD-2X8" device="" value="SSQ-108-03-G-D"/>
 <part name="IC1" library="openblw" deviceset="VR_1OUT" device="XX" value="V7805-1000"/>
 <part name="GND9" library="supply" deviceset="GND" device=""/>
@@
 <part name="FB1" library="resistor" deviceset="L-EU" device="L5650M" value="HR2220V801R-10"/>
 <part name="C16" library="resistor" deviceset="C-EU" device="C0402" value="1u"/>
-<part name="R18" library="resistor" deviceset="R-EU_" device="R0402" value="1K"/>
+<part name="R18" library="resistor" deviceset="R-EU_" device="R0402" value="1k"/>
 <part name="C17" library="resistor" deviceset="C-EU" device="C0402" value="10n"/>
 <part name="GND26" library="supply" deviceset="GND" device=""/>
@@
 <part name="L3" library="openblw" deviceset="SRP1250A" device="" value="SRP1245A-100M"/>
 <part name="FB4" library="resistor" deviceset="L-EU" device="L5650M" value="HR2220V801R-10"/>
-<part name="JP2" library="pinhead" deviceset="PINHD-2X3" device="" value="M20-9980346"/>
-<part name="JP3" library="pinhead" deviceset="PINHD-2X3" device="" value="M20-9980346"/>
+<part name="JP2" library="pinhead" deviceset="PINHD-2X3" device="" value="M20-9980345"/>
+<part name="JP3" library="pinhead" deviceset="PINHD-2X3" device="" value="M20-9980345"/>
 <part name="V7" library="supply" deviceset="+3V3" device=""/>
 <part name="GND11" library="supply" deviceset="GND" device=""/>
@@
 <part name="C41" library="resistor" deviceset="C-EU" device="C0603" value="10u"/>
 <part name="GND46" library="supply1" deviceset="GND" device=""/>
-<part name="C42" library="resistor" deviceset="C-EU" device="C0603" value="1u"/>
+<part name="C42" library="resistor" deviceset="C-EU" device="C0402" value="1u"/>
 <part name="C43" library="resistor" deviceset="C-EU" device="C0402" value="100n"/>
 <part name="GND47" library="supply1" deviceset="GND" device=""/>
@@
 <part name="C45" library="resistor" deviceset="C-EU" device="C0402" value="20p"/>
 <part name="R19" library="resistor" deviceset="R-EU_" device="R0402" value="1M"/>
-<part name="Q6" library="raspi" deviceset="CTS_32X25_SMD" device=""/>
+<part name="Q6" library="raspi" deviceset="CTS_32X25_SMD" device="" value="FA-238 25.0000MB"/>
 <part name="GND53" library="supply1" deviceset="GND" device=""/>
 <part name="U2" library="invensense" deviceset="MPU-9250" device=""/>
 <part name="GND6" library="SparkFun-Aesthetics" deviceset="GND" device=""/>
-<part name="C3" library="SparkFun-Capacitors" deviceset="CAP" device="0603-CAP" value="1uF"/>
-<part name="JP6" library="openblw" deviceset="USB-ID" device="MICRO"/>
+<part name="C3" library="resistor" deviceset="C-EU" device="C0402" value="1uF"/>
+<part name="JP6" library="openblw" deviceset="USB-ID" device="MICRO" value="10118192-0001LF"/>
 <part name="GND8" library="supply1" deviceset="GND" device=""/>
 <part name="P+1" library="supply1" deviceset="+5V" device=""/>
-<part name="JP4" library="pinhead" deviceset="PINHD-2X3" device=""/>
+<part name="JP4" library="pinhead" deviceset="PINHD-2X3" device="" value="M20-9980345"/>
 <part name="LED3" library="led" deviceset="LED" device="CHIP-LED0603" value="GREEN"/>
 <part name="R15" library="resistor" deviceset="R-EU_" device="R0402" value="470R"/>
@@
 <instance part="U2" gate="G$1" x="195.58" y="132.08"/>
 <instance part="GND6" gate="1" x="231.14" y="96.52"/>
-<instance part="C3" gate="G$1" x="167.64" y="124.46" rot="R90"/>
+<instance part="C3" gate="G$1" x="165.1" y="124.46" rot="R90"/>
 <instance part="JP4" gate="A" x="358.14" y="149.86" rot="R90"/>
 <instance part="LED3" gate="G$1" x="81.28" y="111.76" rot="R180"/>

Commit message: before hdmi
Parts:
- removed R9: 10k, resistor:R-EU_R0402
- removed U$7: 282836-2, openblw:282836-2
- added JP5: (no value), openblw:PINHD-1X2
- JP1: device pinhead:PINHD-2X8 -> pinhead:PINHD-2X10
- R8: value 0 -> 12k
Connections:
- removed net N$10: JP1.14, R8.2
- new net N$13: JP3.2, R15.2
- net +12V: no longer U$7.CON01
- net +3V3: now also JP1.18, R8.1; no longer JP1.2, R9.2
- net GND: no longer JP3.2, R15.2, U$7.CON02
- net LAN_RUN: now also R8.2; no longer R8.1, R9.1
- net USB_D_N: now also JP5.2
- net USB_D_P: now also JP5.1
Changed lines of the file:
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@@
 <part name="H3" library="holes" deviceset="MOUNT-PAD-ROUND" device="2.8"/>
 <part name="H4" library="holes" deviceset="MOUNT-PAD-ROUND" device="2.8"/>
-<part name="JP1" library="pinhead" deviceset="PINHD-2X8" device="" value="SSQ-108-03-G-D"/>
+<part name="JP1" library="pinhead" deviceset="PINHD-2X10" device="" value="SSQ-108-03-G-D"/>
 <part name="IC1" library="openblw" deviceset="VR_1OUT" device="XX" value="V7805-1000"/>
 <part name="GND9" library="supply" deviceset="GND" device=""/>
@@
 <part name="GND4" library="supply" deviceset="GND" device=""/>
 <part name="V5" library="supply" deviceset="+12V" device=""/>
-<part name="U$7" library="openblw" deviceset="282836-2" device=""/>
 <part name="U$8" library="openblw" deviceset="282836-2" device=""/>
 <part name="GND13" library="supply" deviceset="GND" device=""/>
@@
 <part name="V4" library="supply" deviceset="+12V" device=""/>
 <part name="GND10" library="supply" deviceset="GND" device=""/>
-<part name="R8" library="resistor" deviceset="R-EU_" device="R0402" value="0"/>
-<part name="R9" library="resistor" deviceset="R-EU_" device="R0402" value="10k"/>
 <part name="K2" library="Wuerth_Elektronik_eiCan_Communication_Connectors_v2.2" deviceset="61400826021" device=""/>
+<part name="JP5" library="openblw" deviceset="PINHD-1X2" device=""/>
+<part name="R8" library="resistor" deviceset="R-EU_" device="R0402" value="12k"/>
 </parts>
 <sheets>
@@
 <instance part="H3" gate="G$1" x="25.4" y="60.96"/>
 <instance part="H4" gate="G$1" x="25.4" y="55.88"/>
-<instance part="JP1" gate="A" x="325.12" y="152.4" rot="MR270"/>
+<instance part="JP1" gate="A" x="327.66" y="152.4" rot="MR270"/>
 <instance part="IC1" gate="A" x="299.72" y="215.9" smashed="yes">
 <attribute name="NAME" x="302.26" y="208.28" size="1.778" layer="95"/>
@@
 <instance part="C2" gate="G$1" x="228.6" y="63.5"/>
 <instance part="V5" gate="1" x="215.9" y="83.82"/>
-<instance part="U$7" gate="G$1" x="165.1" y="33.02" rot="R180"/>
 <instance part="U$8" gate="G$1" x="165.1" y="63.5" rot="R180"/>
 <instance part="GND13" gate="1" x="322.58" y="175.26" rot="R180"/>
@@
 <instance part="V4" gate="1" x="190.5" y="68.58"/>
 <instance part="GND10" gate="1" x="132.08" y="10.16"/>
-<instance part="R8" gate="G$1" x="332.74" y="134.62" rot="R90"/>
-<instance part="R9" gate="G$1" x="342.9" y="127"/>
 </instances>
 <busses>
@@
 <pinref part="R5" gate="G$1" pin="2"/>
 <wire x1="101.6" y1="129.54" x2="101.6" y2="132.08" width="0.1524" layer="91"/>
-<wire x1="101.6" y1="132.08" x2="76.2" y2="132.08" width="0.1524" layer="91"/>
-<pinref part="R15" gate="G$1" pin="2"/>
-<wire x1="76.2" y1="132.08" x2="58.42" y2="132.08" width="0.1524" layer="91"/>
-<wire x1="81.28" y1="129.54" x2="76.2" y2="129.54" width="0.1524" layer="91"/>
-<wire x1="76.2" y1="129.54" x2="76.2" y2="109.22" width="0.1524" layer="91"/>
-<pinref part="JP3" gate="A" pin="2"/>
-<wire x1="76.2" y1="109.22" x2="73.66" y2="109.22" width="0.1524" layer="91"/>
-<wire x1="76.2" y1="132.08" x2="76.2" y2="129.54" width="0.1524" layer="91"/>
-<junction x="76.2" y="132.08"/>
-<junction x="76.2" y="129.54"/>
+<wire x1="101.6" y1="132.08" x2="58.42" y2="132.08" width="0.1524" layer="91"/>
 </segment>
 <segment>
@@
 <segment>
 <pinref part="GND10" gate="1" pin="GND"/>
-<wire x1="162.56" y1="15.24" x2="132.08" y2="15.24" width="0.1524" layer="91"/>
-<wire x1="132.08" y1="15.24" x2="132.08" y2="12.7" width="0.1524" layer="91"/>
 <wire x1="162.56" y1="48.26" x2="132.08" y2="48.26" width="0.1524" layer="91"/>
-<wire x1="132.08" y1="48.26" x2="132.08" y2="15.24" width="0.1524" layer="91"/>
-<junction x="132.08" y="15.24"/>
+<wire x1="132.08" y1="48.26" x2="132.08" y2="12.7" width="0.1524" layer="91"/>
 <pinref part="U$8" gate="G$1" pin="CON02"/>
 <wire x1="162.56" y1="48.26" x2="162.56" y2="53.34" width="0.1524" layer="91"/>
-<pinref part="U$7" gate="G$1" pin="CON02"/>
-<wire x1="162.56" y1="15.24" x2="162.56" y2="22.86" width="0.1524" layer="91"/>
 </segment>
 </net>
@@
 <pinref part="V4" gate="1" pin="+12V"/>
 <wire x1="190.5" y1="48.26" x2="190.5" y2="66.04" width="0.1524" layer="91"/>
-<wire x1="167.64" y1="15.24" x2="190.5" y2="15.24" width="0.1524" layer="91"/>
-<wire x1="190.5" y1="15.24" x2="190.5" y2="48.26" width="0.1524" layer="91"/>
-<junction x="190.5" y="48.26"/>
 <pinref part="U$8" gate="G$1" pin="CON01"/>
 <wire x1="167.64" y1="48.26" x2="167.64" y2="53.34" width="0.1524" layer="91"/>
-<pinref part="U$7" gate="G$1" pin="CON01"/>
-<wire x1="167.64" y1="15.24" x2="167.64" y2="22.86" width="0.1524" layer="91"/>
 </segment>
 </net>
@@
 </segment>
 <segment>
-<label x="317.5" y="114.3" size="1.778" layer="95" rot="R270" xref="yes"/>
-<wire x1="317.5" y1="114.3" x2="317.5" y2="121.92" width="0.1524" layer="91"/>
-<pinref part="JP1" gate="A" pin="2"/>
-<wire x1="317.5" y1="121.92" x2="317.5" y2="147.32" width="0.1524" layer="91"/>
-<wire x1="317.5" y1="121.92" x2="347.98" y2="121.92" width="0.1524" layer="91"/>
-<junction x="317.5" y="121.92"/>
-<pinref part="R9" gate="G$1" pin="2"/>
-<wire x1="347.98" y1="121.92" x2="347.98" y2="127" width="0.1524" layer="91"/>
+<label x="337.82" y="114.3" size="1.778" layer="95" rot="R270" xref="yes"/>
+<pinref part="JP1" gate="A" pin="18"/>
+<wire x1="337.82" y1="147.32" x2="337.82" y2="114.3" width="0.1524" layer="91"/>
 </segment>
 <segment>
@@
 </segment>
 </net>
-<net name="LAN_RUN" class="0">
-<segment>
-<label x="332.74" y="114.3" size="1.778" layer="95" rot="R270" xref="yes"/>
-<pinref part="R8" gate="G$1" pin="1"/>
-<wire x1="332.74" y1="114.3" x2="332.74" y2="127" width="0.1524" layer="91"/>
-<pinref part="R9" gate="G$1" pin="1"/>
-<wire x1="332.74" y1="127" x2="332.74" y2="129.54" width="0.1524" layer="91"/>
-<wire x1="337.82" y1="127" x2="332.74" y2="127" width="0.1524" layer="91"/>
-<junction x="332.74" y="127"/>
-</segment>
-</net>
-<net name="N$10" class="0">
-<segment>
-<pinref part="R8" gate="G$1" pin="2"/>
-<pinref part="JP1" gate="A" pin="14"/>
-<wire x1="332.74" y1="139.7" x2="332.74" y2="147.32" width="0.1524" layer="91"/>
+<net name="N$13" class="1">
+<segment>
+<pinref part="JP3" gate="A" pin="2"/>
+<pinref part="R15" gate="G$1" pin="2"/>
+<wire x1="81.28" y1="129.54" x2="76.2" y2="129.54" width="0.1524" layer="91"/>
+<wire x1="76.2" y1="129.54" x2="76.2" y2="109.22" width="0.1524" layer="91"/>
+<wire x1="76.2" y1="109.22" x2="73.66" y2="109.22" width="0.1524" layer="91"/>
 </segment>
 </net>
@@
 <instance part="P+1" gate="1" x="177.8" y="119.38" rot="R270"/>
 <instance part="K2" gate="G$1" x="264.16" y="50.8" rot="MR270"/>
+<instance part="JP5" gate="G$1" x="175.26" y="109.22" rot="R270"/>
+<instance part="R8" gate="G$1" x="314.96" y="63.5" rot="R90"/>
 </instances>
 <busses>
@@
 <wire x1="287.02" y1="91.44" x2="287.02" y2="81.28" width="0.1524" layer="91"/>
 <wire x1="287.02" y1="81.28" x2="304.8" y2="81.28" width="0.1524" layer="91"/>
-<wire x1="304.8" y1="81.28" x2="304.8" y2="71.12" width="0.1524" layer="91"/>
-<label x="304.8" y="71.12" size="1.778" layer="95" rot="R270" xref="yes"/>
+<wire x1="304.8" y1="81.28" x2="304.8" y2="73.66" width="0.1524" layer="91"/>
+<label x="304.8" y="53.34" size="1.778" layer="95" rot="R270" xref="yes"/>
+<pinref part="R8" gate="G$1" pin="2"/>
+<wire x1="304.8" y1="73.66" x2="304.8" y2="53.34" width="0.1524" layer="91"/>
+<wire x1="314.96" y1="68.58" x2="314.96" y2="73.66" width="0.1524" layer="91"/>
+<wire x1="314.96" y1="73.66" x2="304.8" y2="73.66" width="0.1524" layer="91"/>
+<junction x="304.8" y="73.66"/>
 </segment>
 </net>
@@
 <segment>
 <pinref part="IC6" gate="G$1" pin="USBDM0"/>
-<wire x1="238.76" y1="127" x2="162.56" y2="127" width="0.1524" layer="91"/>
+<wire x1="238.76" y1="127" x2="175.26" y2="127" width="0.1524" layer="91"/>
 <label x="152.4" y="127" size="1.778" layer="95" rot="R180" xref="yes"/>
 <pinref part="JP6" gate="G$1" pin="D-"/>
+<wire x1="175.26" y1="127" x2="162.56" y2="127" width="0.1524" layer="91"/>
 <wire x1="162.56" y1="127" x2="152.4" y2="127" width="0.1524" layer="91"/>
 <wire x1="162.56" y1="116.84" x2="162.56" y2="127" width="0.1524" layer="91"/>
 <junction x="162.56" y="127"/>
+<pinref part="JP5" gate="G$1" pin="2"/>
+<wire x1="175.26" y1="111.76" x2="175.26" y2="127" width="0.1524" layer="91"/>
+<junction x="175.26" y="127"/>
 </segment>
 </net>
@@
 <segment>
 <pinref part="IC6" gate="G$1" pin="USBDP0"/>
-<wire x1="238.76" y1="124.46" x2="165.1" y2="124.46" width="0.1524" layer="91"/>
+<wire x1="238.76" y1="124.46" x2="177.8" y2="124.46" width="0.1524" layer="91"/>
 <label x="152.4" y="124.46" size="1.778" layer="95" rot="R180" xref="yes"/>
 <pinref part="JP6" gate="G$1" pin="D+"/>
+<wire x1="177.8" y1="124.46" x2="165.1" y2="124.46" width="0.1524" layer="91"/>
 <wire x1="165.1" y1="124.46" x2="152.4" y2="124.46" width="0.1524" layer="91"/>
 <wire x1="165.1" y1="116.84" x2="165.1" y2="124.46" width="0.1524" layer="91"/>
 <junction x="165.1" y="124.46"/>
+<pinref part="JP5" gate="G$1" pin="1"/>
+<wire x1="177.8" y1="111.76" x2="177.8" y2="124.46" width="0.1524" layer="91"/>
+<junction x="177.8" y="124.46"/>
 </segment>
 </net>
@@
 <label x="355.6" y="137.16" size="1.778" layer="95" rot="R90" xref="yes"/>
 </segment>
-</net>
+<segment>
+<label x="314.96" y="53.34" size="1.778" layer="95" rot="R270" xref="yes"/>
+<pinref part="R8" gate="G$1" pin="1"/>
+<wire x1="314.96" y1="53.34" x2="314.96" y2="58.42" width="0.1524" layer="91"/>
+</segment>
+</net>
