File: interface_board/interface_board.sch (EAGLE design)
At the start: 86 parts, among them IC1 V7805-1000, IC6 LAN9512-JZX, K2 61400826021, Q1 IRLML6346TRPBF, Q6 FA-238 25.0000MB, U1 AL5812MP-13, U2 MPU-9250

Commit message: before autorouter
Parts:
- added C5, C6: 22u, resistor:C-EUC0603
- added L1: SRN4018-100M(10u), openblw:BOURNS-SRN4018
- C16: value 1u -> 10u; device resistor:C-EUC0402 -> resistor:C-EUC0603
Connections:
- new net N$10: C5.1, IC1.OUT, L1.2
- net +12V: now also U$4.CON01; no longer U$4.CON02
- net +5V: now also C6.1, L1.1; no longer IC1.OUT
- net GND: now also C5.2, C6.2, JP1.19, U$4.CON02; no longer U$4.CON01
Other:
- moved on the sheet: C16, IC1
Changed lines of the file:
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@@
 <part name="V9" library="supply" deviceset="+12V" device=""/>
 <part name="FB1" library="resistor" deviceset="L-EU" device="L5650M" value="HR2220V801R-10"/>
-<part name="C16" library="resistor" deviceset="C-EU" device="C0402" value="1u"/>
+<part name="C16" library="resistor" deviceset="C-EU" device="C0603" value="10u"/>
 <part name="R18" library="resistor" deviceset="R-EU_" device="R0402" value="1k"/>
 <part name="C17" library="resistor" deviceset="C-EU" device="C0402" value="10n"/>
 <part name="GND26" library="supply" deviceset="GND" device=""/>
-<part name="GND30" library="supply" deviceset="GND" device=""/>
 <part name="U$2" library="openblw" deviceset="282836-2" device=""/>
 <part name="L3" library="openblw" deviceset="SRP1250A" device="" value="SRP1245A-100M"/>
@@
 <part name="JP5" library="openblw" deviceset="PINHD-1X2" device=""/>
 <part name="R8" library="resistor" deviceset="R-EU_" device="R0402" value="12k"/>
+<part name="C5" library="resistor" deviceset="C-EU" device="C0603" value="22u"/>
+<part name="C6" library="resistor" deviceset="C-EU" device="C0603" value="22u"/>
+<part name="L1" library="openblw" deviceset="BOURNS-SRN4018" device="" value="SRN4018-100M(10u)"/>
 </parts>
 <sheets>
@@
 <instance part="H4" gate="G$1" x="25.4" y="55.88"/>
 <instance part="JP1" gate="A" x="327.66" y="152.4" rot="MR270"/>
-<instance part="IC1" gate="A" x="299.72" y="215.9" smashed="yes">
-<attribute name="NAME" x="302.26" y="208.28" size="1.778" layer="95"/>
-<attribute name="VALUE" x="292.1" y="220.98" size="1.778" layer="96"/>
+<instance part="IC1" gate="A" x="271.78" y="215.9" smashed="yes">
+<attribute name="NAME" x="274.32" y="208.28" size="1.778" layer="95"/>
+<attribute name="VALUE" x="264.16" y="220.98" size="1.778" layer="96"/>
 </instance>
 <instance part="GND9" gate="1" x="226.06" y="223.52" rot="R90"/>
-<instance part="V1" gate="1" x="309.88" y="226.06"/>
-<instance part="GND14" gate="1" x="299.72" y="198.12"/>
+<instance part="V1" gate="1" x="322.58" y="226.06"/>
+<instance part="GND14" gate="1" x="271.78" y="198.12"/>
 <instance part="V9" gate="1" x="256.54" y="226.06"/>
 <instance part="FB1" gate="G$1" x="213.36" y="215.9" rot="R90"/>
-<instance part="C16" gate="G$1" x="248.92" y="210.82"/>
+<instance part="C16" gate="G$1" x="256.54" y="210.82"/>
 <instance part="R18" gate="G$1" x="223.52" y="208.28" rot="R270"/>
 <instance part="C17" gate="G$1" x="223.52" y="198.12"/>
 <instance part="GND26" gate="1" x="223.52" y="187.96"/>
-<instance part="GND30" gate="1" x="248.92" y="198.12"/>
 <instance part="U$2" gate="G$1" x="195.58" y="200.66" rot="MR0"/>
 <instance part="L3" gate="G$1" x="236.22" y="215.9"/>
@@
 <instance part="GND11" gate="1" x="58.42" y="137.16" rot="R180"/>
 <instance part="V3" gate="1" x="63.5" y="236.22"/>
-<instance part="U$4" gate="G$1" x="38.1" y="218.44"/>
+<instance part="U$4" gate="G$1" x="38.1" y="218.44" rot="MR0"/>
 <instance part="GND4" gate="1" x="35.56" y="241.3" rot="R180"/>
 <instance part="GND5" gate="1" x="254" y="58.42"/>
@@
 <instance part="V4" gate="1" x="190.5" y="68.58"/>
 <instance part="GND10" gate="1" x="132.08" y="10.16"/>
+<instance part="C5" gate="G$1" x="281.94" y="210.82"/>
+<instance part="C6" gate="G$1" x="320.04" y="210.82"/>
+<instance part="L1" gate="G$1" x="302.26" y="215.9"/>
 </instances>
 <busses>
@@
 </segment>
 <segment>
-<pinref part="IC1" gate="A" pin="GND"/>
-<pinref part="GND14" gate="1" pin="GND"/>
-<wire x1="299.72" y1="208.28" x2="299.72" y2="200.66" width="0.1524" layer="91"/>
-</segment>
-<segment>
 <pinref part="GND26" gate="1" pin="GND"/>
 <pinref part="C17" gate="G$1" pin="2"/>
@@
 </segment>
 <segment>
-<pinref part="GND30" gate="1" pin="GND"/>
 <pinref part="C16" gate="G$1" pin="2"/>
-<wire x1="248.92" y1="200.66" x2="248.92" y2="205.74" width="0.1524" layer="91"/>
+<pinref part="IC1" gate="A" pin="GND"/>
+<pinref part="GND14" gate="1" pin="GND"/>
+<wire x1="256.54" y1="203.2" x2="256.54" y2="205.74" width="0.1524" layer="91"/>
+<wire x1="271.78" y1="208.28" x2="271.78" y2="203.2" width="0.1524" layer="91"/>
+<pinref part="C5" gate="G$1" pin="2"/>
+<wire x1="271.78" y1="203.2" x2="271.78" y2="200.66" width="0.1524" layer="91"/>
+<wire x1="281.94" y1="205.74" x2="281.94" y2="203.2" width="0.1524" layer="91"/>
+<wire x1="281.94" y1="203.2" x2="271.78" y2="203.2" width="0.1524" layer="91"/>
+<junction x="271.78" y="203.2"/>
+<pinref part="C6" gate="G$1" pin="2"/>
+<wire x1="320.04" y1="205.74" x2="320.04" y2="203.2" width="0.1524" layer="91"/>
+<wire x1="320.04" y1="203.2" x2="281.94" y2="203.2" width="0.1524" layer="91"/>
+<junction x="281.94" y="203.2"/>
+<wire x1="256.54" y1="203.2" x2="271.78" y2="203.2" width="0.1524" layer="91"/>
 </segment>
 <segment>
@@
 </segment>
 <segment>
-<pinref part="U$4" gate="G$1" pin="CON01"/>
 <pinref part="GND4" gate="1" pin="GND"/>
-<wire x1="35.56" y1="228.6" x2="35.56" y2="238.76" width="0.1524" layer="91"/>
+<pinref part="U$4" gate="G$1" pin="CON02"/>
+<wire x1="35.56" y1="238.76" x2="35.56" y2="228.6" width="0.1524" layer="91"/>
 </segment>
 <segment>
@@
 <wire x1="332.74" y1="160.02" x2="322.58" y2="160.02" width="0.1524" layer="91"/>
 <junction x="322.58" y="160.02"/>
+<pinref part="JP1" gate="A" pin="19"/>
+<wire x1="340.36" y1="154.94" x2="340.36" y2="160.02" width="0.1524" layer="91"/>
+<wire x1="340.36" y1="160.02" x2="332.74" y2="160.02" width="0.1524" layer="91"/>
+<junction x="332.74" y="160.02"/>
 </segment>
 <segment>
@@
 <net name="+5V" class="5">
 <segment>
-<pinref part="IC1" gate="A" pin="OUT"/>
 <pinref part="V1" gate="1" pin="+5V"/>
-<wire x1="307.34" y1="215.9" x2="309.88" y2="215.9" width="0.1524" layer="91"/>
-<wire x1="309.88" y1="215.9" x2="309.88" y2="223.52" width="0.1524" layer="91"/>
+<wire x1="320.04" y1="215.9" x2="322.58" y2="215.9" width="0.1524" layer="91"/>
+<wire x1="322.58" y1="215.9" x2="322.58" y2="223.52" width="0.1524" layer="91"/>
+<pinref part="C6" gate="G$1" pin="1"/>
+<wire x1="320.04" y1="213.36" x2="320.04" y2="215.9" width="0.1524" layer="91"/>
+<pinref part="L1" gate="G$1" pin="1"/>
+<wire x1="309.88" y1="215.9" x2="320.04" y2="215.9" width="0.1524" layer="91"/>
+<junction x="320.04" y="215.9"/>
 </segment>
 <segment>
@@
 <net name="+12V" class="5">
 <segment>
-<wire x1="241.3" y1="215.9" x2="248.92" y2="215.9" width="0.1524" layer="91"/>
+<wire x1="241.3" y1="215.9" x2="256.54" y2="215.9" width="0.1524" layer="91"/>
 <pinref part="C16" gate="G$1" pin="1"/>
-<wire x1="248.92" y1="215.9" x2="256.54" y2="215.9" width="0.1524" layer="91"/>
-<wire x1="248.92" y1="213.36" x2="248.92" y2="215.9" width="0.1524" layer="91"/>
-<junction x="248.92" y="215.9"/>
+<wire x1="256.54" y1="213.36" x2="256.54" y2="215.9" width="0.1524" layer="91"/>
+<junction x="256.54" y="215.9"/>
 <pinref part="V9" gate="1" pin="+12V"/>
 <wire x1="256.54" y1="223.52" x2="256.54" y2="215.9" width="0.1524" layer="91"/>
@@
 <pinref part="L3" gate="G$1" pin="2"/>
 <pinref part="IC1" gate="A" pin="IN"/>
-<wire x1="256.54" y1="215.9" x2="292.1" y2="215.9" width="0.1524" layer="91"/>
+<wire x1="256.54" y1="215.9" x2="264.16" y2="215.9" width="0.1524" layer="91"/>
 </segment>
 <segment>
@@
 <wire x1="63.5" y1="231.14" x2="63.5" y2="233.68" width="0.1524" layer="91"/>
 <junction x="63.5" y="231.14"/>
-<pinref part="U$4" gate="G$1" pin="CON02"/>
-<wire x1="40.64" y1="228.6" x2="40.64" y2="231.14" width="0.1524" layer="91"/>
 <wire x1="40.64" y1="231.14" x2="63.5" y2="231.14" width="0.1524" layer="91"/>
+<pinref part="U$4" gate="G$1" pin="CON01"/>
+<wire x1="40.64" y1="231.14" x2="40.64" y2="228.6" width="0.1524" layer="91"/>
 </segment>
 <segment>
@@
 </segment>
 </net>
+<net name="N$10" class="5">
+<segment>
+<pinref part="IC1" gate="A" pin="OUT"/>
+<wire x1="279.4" y1="215.9" x2="281.94" y2="215.9" width="0.1524" layer="91"/>
+<pinref part="C5" gate="G$1" pin="1"/>
+<wire x1="281.94" y1="213.36" x2="281.94" y2="215.9" width="0.1524" layer="91"/>
+<pinref part="L1" gate="G$1" pin="2"/>
+<wire x1="281.94" y1="215.9" x2="294.64" y2="215.9" width="0.1524" layer="91"/>
+<junction x="281.94" y="215.9"/>
+</segment>
+</net>

Commit message: interface board 0.7 rpcm board 0.10
Parts:
- removed JP5: (no value), openblw:PINHD-1X2
- removed U$8: 282836-2, openblw:282836-2
- added C11, C7: 4.7n, resistor:C-EUC0402
- added R11, R9: 1M, resistor:R-EU_R0402
- K2: device Wuerth_Elektronik_eiCan_Communication_Connectors_v2.2:61400826021 -> openblw:61400826021
Connections:
- net N$43 renamed AVDD18PLL
- new net PWMC: JP1.14, JP4.3
- new net PWMD: JP1.15, JP4.5
- new net USB1_SHELL: C7.1, K2.SHELL@1, K2.SHELL@2, K2.SHELL@3, K2.SHELL@4, R9.1
- new net USB2_SHELL: C11.1, JP6.SHELL, R11.1
- net +12V: no longer U$8.CON01
- net +3V3: now also JP1.2
- net GND: now also C11.2, C7.2, R11.2, R9.2; no longer U$8.CON02
- net USB_D_N: no longer JP5.2
- net USB_D_P: no longer JP5.1
