File: camera_unit/camera_unit.sch (EAGLE design)
At the start: 2 parts, among them U1 DF37-30D-0.4V, U2 DF37*-30D*-0.4VHEADER

Commit message: camera_unit, camera_adapter
Parts:
- removed U1: DF37-30D-0.4V, openblw:DF37-30D-0.4V
- removed U2: DF37*-30D*-0.4VHEADER, openblw:DF37-30D-0.4VHEADER
Connections:
- removed net N$1: U1.2, U2.2
- removed net N$10: U1.20, U2.20
- removed net N$11: U1.22, U2.22
- removed net N$12: U1.24, U2.24
- removed net N$13: U1.26, U2.26
- removed net N$14: U1.28, U2.28
- removed net N$15: U1.30, U2.30
- removed net N$16: U1.1, U2.1
- removed net N$17: U1.3, U2.3
- removed net N$18: U1.5, U2.5
- removed net N$19: U1.7, U2.7
- removed net N$2: U1.4, U2.4
- removed net N$20: U1.9, U2.9
- removed net N$21: U1.11, U2.11
- removed net N$22: U1.13, U2.13
- removed net N$23: U1.15, U2.15
- removed net N$24: U1.29, U2.29
- removed net N$25: U1.27, U2.27
- removed net N$26: U1.25, U2.25
- removed net N$27: U1.23, U2.23
- removed net N$28: U1.21, U2.21
- removed net N$29: U1.19, U2.19
- removed net N$3: U1.6, U2.6
- removed net N$30: U1.17, U2.17
- removed net N$4: U1.8, U2.8
- removed net N$5: U1.10, U2.10
- removed net N$6: U1.12, U2.12
- removed net N$7: U1.14, U2.14
- removed net N$8: U1.16, U2.16
- removed net N$9: U1.18, U2.18
