File: usb_ext_board/usb_ext_board.brd (EAGLE design)
At the start: 10 x 28.5 mm, 2 parts

Commit message: debug
Parts:
- moved MALE1 2.00 mm to (5.00, 27.5)
Routing:
- net ID: track 22.5 -> 24.5 mm
- net D-: track 22.5 -> 24.5 mm
- net D+: track 22.5 -> 24.5 mm
Other:
- board size 10 x 28.5 mm -> 10 x 30.5 mm
- board text added: "11.0mm 1.6mm 10.0mm 1.6mm margin:0.3mm total:24.5mm"
Changed lines of the file:
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@@
 <layer number="27" name="tValues" color="7" fill="1" visible="yes" active="yes"/>
 <layer number="28" name="bValues" color="7" fill="1" visible="yes" active="yes"/>
-<layer number="29" name="tStop" color="7" fill="3" visible="no" active="yes"/>
-<layer number="30" name="bStop" color="7" fill="6" visible="no" active="yes"/>
-<layer number="31" name="tCream" color="7" fill="4" visible="no" active="yes"/>
-<layer number="32" name="bCream" color="7" fill="5" visible="no" active="yes"/>
-<layer number="33" name="tFinish" color="6" fill="3" visible="no" active="yes"/>
-<layer number="34" name="bFinish" color="6" fill="6" visible="no" active="yes"/>
-<layer number="35" name="tGlue" color="7" fill="4" visible="no" active="yes"/>
-<layer number="36" name="bGlue" color="7" fill="5" visible="no" active="yes"/>
-<layer number="37" name="tTest" color="7" fill="1" visible="no" active="yes"/>
-<layer number="38" name="bTest" color="7" fill="1" visible="no" active="yes"/>
+<layer number="29" name="tStop" color="7" fill="3" visible="yes" active="yes"/>
+<layer number="30" name="bStop" color="7" fill="6" visible="yes" active="yes"/>
+<layer number="31" name="tCream" color="7" fill="4" visible="yes" active="yes"/>
+<layer number="32" name="bCream" color="7" fill="5" visible="yes" active="yes"/>
+<layer number="33" name="tFinish" color="6" fill="3" visible="yes" active="yes"/>
+<layer number="34" name="bFinish" color="6" fill="6" visible="yes" active="yes"/>
+<layer number="35" name="tGlue" color="7" fill="4" visible="yes" active="yes"/>
+<layer number="36" name="bGlue" color="7" fill="5" visible="yes" active="yes"/>
+<layer number="37" name="tTest" color="7" fill="1" visible="yes" active="yes"/>
+<layer number="38" name="bTest" color="7" fill="1" visible="yes" active="yes"/>
 <layer number="39" name="tKeepout" color="4" fill="11" visible="yes" active="yes"/>
 <layer number="40" name="bKeepout" color="1" fill="11" visible="yes" active="yes"/>
@@
 <layer number="42" name="bRestrict" color="1" fill="10" visible="yes" active="yes"/>
 <layer number="43" name="vRestrict" color="2" fill="10" visible="yes" active="yes"/>
-<layer number="44" name="Drills" color="7" fill="1" visible="no" active="yes"/>
-<layer number="45" name="Holes" color="7" fill="1" visible="no" active="yes"/>
-<layer number="46" name="Milling" color="3" fill="1" visible="no" active="yes"/>
-<layer number="47" name="Measures" color="7" fill="1" visible="no" active="yes"/>
+<layer number="44" name="Drills" color="7" fill="1" visible="yes" active="yes"/>
+<layer number="45" name="Holes" color="7" fill="1" visible="yes" active="yes"/>
+<layer number="46" name="Milling" color="3" fill="1" visible="yes" active="yes"/>
+<layer number="47" name="Measures" color="7" fill="1" visible="yes" active="yes"/>
 <layer number="48" name="Document" color="7" fill="1" visible="yes" active="yes"/>
 <layer number="49" name="Reference" color="7" fill="1" visible="yes" active="yes"/>
@@
 <plain>
 <wire x1="0" y1="0" x2="10" y2="0" width="0" layer="20"/>
-<wire x1="10" y1="0" x2="10" y2="28.5" width="0" layer="20"/>
-<wire x1="10" y1="28.5" x2="0" y2="28.5" width="0" layer="20"/>
-<wire x1="0" y1="28.5" x2="0" y2="0" width="0" layer="20"/>
+<wire x1="10" y1="0" x2="10" y2="30.5" width="0" layer="20"/>
+<wire x1="10" y1="30.5" x2="0" y2="30.5" width="0" layer="20"/>
+<wire x1="0" y1="30.5" x2="0" y2="0" width="0" layer="20"/>
+<text x="18.4" y="24.4" size="1.778" layer="48">11.0mm
+ 1.6mm
+10.0mm
+ 1.6mm
+margin:0.3mm
+total:24.5mm</text>
 </plain>
 <attributes>
@@
 </autorouter>
 <elements>
-<element name="MALE1" library="openblw" package="USB3150-30-130" value="USB-ID" x="5" y="25.5"/>
+<element name="MALE1" library="openblw" package="USB3150-30-130" value="USB-ID" x="5" y="27.5"/>
 <element name="MALE2" library="openblw" package="USB3150-30-130" value="USB-ID" x="5" y="3"/>
 </elements>
@@
 <contactref element="MALE1" pad="ID@4"/>
 <contactref element="MALE2" pad="ID@4"/>
-<wire x1="4.35" y1="25.825" x2="4.35" y2="3.325" width="0.127" layer="1"/>
+<wire x1="4.35" y1="27.825" x2="4.35" y2="3.325" width="0.127" layer="1"/>
 </signal>
 <signal name="D+">
 <contactref element="MALE1" pad="D+@3"/>
 <contactref element="MALE2" pad="D+@3"/>
-<wire x1="5" y1="25.175" x2="5" y2="2.675" width="0.127" layer="1"/>
+<wire x1="5" y1="27.175" x2="5" y2="2.675" width="0.127" layer="1"/>
 </signal>
 <signal name="D-">
 <contactref element="MALE1" pad="D-@2"/>
 <contactref element="MALE2" pad="D-@2"/>
-<wire x1="5.65" y1="25.825" x2="5.65" y2="3.325" width="0.127" layer="1"/>
+<wire x1="5.65" y1="27.825" x2="5.65" y2="3.325" width="0.127" layer="1"/>
 </signal>
 <signal name="VCC">
@@
 <contactref element="MALE2" pad="VCC@1"/>
 <polygon width="0.127" layer="1">
-<vertex x="7.3" y="28.5"/>
+<vertex x="7.3" y="30.2"/>
 <vertex x="7.3" y="0.5"/>
 <vertex x="9.5" y="0.5"/>
-<vertex x="9.6" y="28.5"/>
+<vertex x="9.6" y="30.2"/>
 </polygon>
-<wire x1="6.3" y1="25.175" x2="7.025" y2="25.9" width="0.6096" layer="1"/>
-<wire x1="7.025" y1="25.9" x2="7.4" y2="25.9" width="0.6096" layer="1"/>
+<wire x1="6.3" y1="27.175" x2="6.925" y2="27.8" width="0.6096" layer="1"/>
+<wire x1="6.925" y1="27.8" x2="7.3" y2="27.8" width="0.6096" layer="1"/>
 <wire x1="6.3" y1="2.675" x2="6.925" y2="3.3" width="0.6096" layer="1"/>
 <wire x1="6.925" y1="3.3" x2="7.3" y2="3.3" width="0.6096" layer="1"/>
@@
 <contactref element="MALE2" pad="SHELL@11"/>
 <contactref element="MALE2" pad="SHELL@7"/>
-<polygon width="0.6096" layer="1">
-<vertex x="0" y="28.5"/>
-<vertex x="6.7" y="28.5"/>
+<polygon width="0.254" layer="1">
+<vertex x="0" y="30.5"/>
+<vertex x="6.7" y="30.5"/>
 <vertex x="6.7" y="0"/>
 <vertex x="0" y="0"/>
 </polygon>
 <polygon width="0.254" layer="16">
-<vertex x="10" y="28.5"/>
-<vertex x="0" y="28.5"/>
+<vertex x="10" y="30.5"/>
+<vertex x="0" y="30.5"/>
 <vertex x="0" y="0"/>
 <vertex x="10" y="0"/>
@@
 </board>
 </drawing>
+<compatibility>
+<note version="6.3" minversion="6.2.2" severity="warning">
+Since Version 6.2.2 text objects can contain more than one line,
+which will not be processed correctly with this version.
+</note>
+</compatibility>
 </eagle>

Commit message: after test
Parts:
- added LOGO1: (no value), openblw:OHMYDIGIFAB_LOGO
Routing:
- net GND: track 0.00 -> 3.17 mm
Other:
- board text added: "Picam360"
- board text added: "Rev.0.1"
- board text added: "USB Ext Board"
Changed lines of the file:
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@@
 <?xml version="1.0" encoding="utf-8"?>
 <!DOCTYPE eagle SYSTEM "eagle.dtd">
-<eagle version="7.5.0">
+<eagle version="8.1.1">
 <drawing>
 <settings>
@@
 <layers>
 <layer number="1" name="Top" color="4" fill="1" visible="yes" active="yes"/>
+<layer number="2" name="Route2" color="1" fill="3" visible="yes" active="yes"/>
+<layer number="15" name="Route15" color="4" fill="6" visible="yes" active="yes"/>
 <layer number="16" name="Bottom" color="1" fill="1" visible="yes" active="yes"/>
 <layer number="17" name="Pads" color="2" fill="1" visible="yes" active="yes"/>
@@
 <layer number="56" name="wert" color="7" fill="1" visible="no" active="no"/>
 <layer number="57" name="tCAD" color="7" fill="1" visible="no" active="no"/>
+<layer number="58" name="bCAD" color="7" fill="1" visible="no" active="no"/>
 <layer number="59" name="tCarbon" color="7" fill="1" visible="no" active="no"/>
 <layer number="60" name="bCarbon" color="7" fill="1" visible="no" active="no"/>
@@
 margin:0.3mm
 total:24.5mm</text>
+<text x="3.07" y="5.099" size="2.54" layer="21" rot="R90">Picam360</text>
+<text x="4.868" y="5.199" size="1.4224" layer="21" rot="R90">USB Ext Board</text>
+<text x="6.763" y="5.168" size="1.4224" layer="21" rot="R90">Rev.0.1</text>
 </plain>
 <attributes>
@@
 <element name="MALE1" library="openblw" package="USB3150-30-130" value="USB-ID" x="5" y="27.5"/>
 <element name="MALE2" library="openblw" package="USB3150-30-130" value="USB-ID" x="5" y="3"/>
+<element name="LOGO1" library="openblw" package="OHMYDIGIFAB_LOGO" value="" x="6.713" y="22.57" smashed="yes" rot="R90"/>
 </elements>
 <signals>
@@
 <vertex x="10" y="0"/>
 </polygon>
+<wire x1="3.1" y1="27.775" x2="3.7" y2="27.175" width="0.6096" layer="16"/>
+<wire x1="3.1" y1="27.8" x2="3.1" y2="27.775" width="0.6096" layer="16"/>
+<wire x1="3.7" y1="27.175" x2="3.1" y2="27.775" width="0.6096" layer="1"/>
+<wire x1="3.1" y1="27.775" x2="3.1" y2="27.8" width="0.6096" layer="1"/>
+<wire x1="3.7" y1="2.675" x2="3.3" y2="3.075" width="0.6096" layer="16"/>
+<wire x1="3.3" y1="3.075" x2="3.3" y2="3.1" width="0.6096" layer="16"/>
+<wire x1="3.7" y1="2.675" x2="3.2" y2="3.175" width="0.6096" layer="1"/>
+<wire x1="3.2" y1="3.175" x2="3.2" y2="3.3" width="0.6096" layer="1"/>
 </signal>
 </signals>
