File: nekojara/usb/usb.brd (EAGLE design)
At the start: 13 x 12 mm, 5 parts, among them X1 USBPCB

Commit message: nekojara : usb
Parts:
- flipped JP2 to the top
- flipped JP3 to the top
Changed lines of the file:
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@@
 </autorouter>
 <elements>
-<element name="JP2" library="pinhead+" package="1X01" value="" x="10.922" y="4.699" smashed="yes" rot="MR0">
-<attribute name="VALUE" x="12.192" y="1.524" size="1.27" layer="28" rot="MR0"/>
+<element name="JP2" library="pinhead+" package="1X01" value="" x="10.922" y="4.699" smashed="yes">
+<attribute name="VALUE" x="9.652" y="1.524" size="1.27" layer="27"/>
 </element>
-<element name="JP3" library="pinhead+" package="1X01" value="" x="10.922" y="2.159" smashed="yes" rot="MR0">
-<attribute name="VALUE" x="12.192" y="-1.016" size="1.27" layer="28" rot="MR0"/>
+<element name="JP3" library="pinhead+" package="1X01" value="" x="10.922" y="2.159" smashed="yes">
+<attribute name="VALUE" x="9.652" y="-1.016" size="1.27" layer="27"/>
 </element>
 <element name="X1" library="usb" package="USB-A-PCB" value="USBPCB" x="5" y="6"/>
@@
 <contactref element="X1" pad="USB_P"/>
 <contactref element="JP1" pad="1"/>
-<wire x1="10.922" y1="7.239" x2="10.683" y2="7" width="0.8128" layer="1" curve="-90"/>
-<wire x1="10.683" y1="7" x2="5.3" y2="7" width="0.8128" layer="1"/>
+<wire x1="10.922" y1="7.239" x2="10.683" y2="7" width="1.016" layer="1"/>
+<wire x1="10.683" y1="7" x2="5.3" y2="7" width="1.016" layer="1"/>
 </signal>
 <signal name="USB_N">
 <contactref element="X1" pad="USB_M"/>
 <contactref element="JP2" pad="1"/>
-<wire x1="10.922" y1="4.699" x2="10.621" y2="5" width="0.8128" layer="1" curve="90"/>
-<wire x1="10.621" y1="5" x2="5.3" y2="5" width="0.8128" layer="1"/>
+<wire x1="10.922" y1="4.699" x2="10.621" y2="5" width="1.016" layer="1"/>
+<wire x1="10.621" y1="5" x2="5.3" y2="5" width="1.016" layer="1"/>
 </signal>
 <signal name="5V">
 <contactref element="X1" pad="5V"/>
 <contactref element="JP3" pad="1"/>
-<wire x1="10.922" y1="2.159" x2="10.581" y2="2.5" width="0.8128" layer="1" curve="90"/>
-<wire x1="10.581" y1="2.5" x2="4.8" y2="2.5" width="0.8128" layer="1"/>
+<wire x1="10.922" y1="2.159" x2="10.581" y2="2.5" width="1.016" layer="1"/>
+<wire x1="10.581" y1="2.5" x2="4.8" y2="2.5" width="1.016" layer="1"/>
 </signal>
 <signal name="GND">
 <contactref element="X1" pad="GND"/>
 <contactref element="JP4" pad="1"/>
-<wire x1="10.922" y1="9.779" x2="10.643" y2="9.5" width="0.8128" layer="1" curve="-90"/>
-<wire x1="10.643" y1="9.5" x2="4.8" y2="9.5" width="0.8128" layer="1"/>
 <polygon width="0.2" layer="16">
 <vertex x="0" y="0"/>
@@
 <vertex x="0" y="12"/>
 </polygon>
+<wire x1="10.922" y1="9.779" x2="10.643" y2="9.5" width="0.8128" layer="1"/>
+<wire x1="10.643" y1="9.5" x2="4.8" y2="9.5" width="0.8128" layer="1"/>
 </signal>
 </signals>
