File: nekojara/nekojara_board/nekojara_board.brd (EAGLE design)
At the start: 65 x 56 mm, 19 parts, among them U1 DRV8835, U2 MPU-9250, U3 DRV8835, U4 DRV8835

Commit message: nekojara
Parts:
- added C10, C9: 100n, resistor:C0402
- added C11, C12: 22u, resistor:C0603
- added C16: 10u, resistor:C0603
- added D1: 1N34A, diode:DO07
- added IC1: V7805-1000, openblw:DIP_3PIN
- added J1: (no value), con-jack:SPC4077
- added JP4: (no value), pinhead:1X04M
- added JP5, JP6: (no value), pinhead+:2X03
- added L1: SRN4018-100M(10u), openblw:BOURNS-SRN4018
- added SJ1, SJ2, SJ3, SJ4: SOLDERJUMPERNO, SparkFun-Retired:SJ_2S-NO
- added U5: DRV8835, bt_motordriver:WSON_2X3
- JP1, JP2, JP3: device pinhead:1X04 -> pinhead:1X04M
- PCB1: device e14_Rpi3_RevA:RPI3 -> nekojara_board:RPI3
- moved U4 17.7 mm to (32.5, 10.0)
- moved JP3 17.7 mm to (32.5, 3.50), turned to 180 degrees
- moved C8 17.5 mm to (29.2, 9.02)
- moved C7 17.5 mm to (29.2, 10.9)
- moved JP2 11.4 mm to (22.3, 3.50), turned to 180 degrees
- moved U3 11.3 mm to (22.4, 10.0)
- moved C5 11.0 mm to (18.9, 10.9)
- moved C6 11.0 mm to (18.9, 9.02)
- moved U1 2.53 mm to (12.1, 10.0)
- moved JP1 2.53 mm to (12.1, 3.50), turned to 180 degrees
- moved C1 2.16 mm to (8.76, 10.9)
- moved C2 2.16 mm to (8.76, 9.02)
- moved C4 0.51 mm to (9.78, 43.9)
Connections:
- removed net MD1_MODE: PCB1.P$13, U1.11
- removed net MD2_MODE: PCB1.P$36, U3.11
- removed net MD3_MODE: PCB1.P$35, U4.11
- new net +12V: C10.2, C16.1, C2.2, C6.2, C8.2, D1.C, IC1.IN, J1.3, U1.1, U3.1, U4.1, U5.1
- new net GPIO4: JP6.3, PCB1.P$7
- new net MD4_A1: PCB1.P$37, U5.10
- new net MD4_A2: PCB1.P$13, U5.9
- new net MD4_B1: PCB1.P$36, U5.8
- new net MD4_B2: PCB1.P$35, U5.7
- new net N$14: JP4.3, U5.3
- new net N$15: JP4.2, U5.4
- new net N$16: JP4.1, U5.5
- new net N$17: SJ4.1, U5.11
- new net N$18: SJ3.1, U4.11
- new net N$19: SJ2.1, U3.11
- new net N$20: SJ1.1, U1.11
- new net N$22: C11.1, IC1.OUT, L1.P$2
- new net N$4: JP4.4, U5.2
- new net RX: JP6.5, PCB1.P$10
- new net SPI_CE0_N: JP5.2, PCB1.P$24
- new net SPI_CE1_N: JP5.4, PCB1.P$26
- new net SPI_MISO: JP5.3, PCB1.P$21
- new net SPI_MOSI: JP5.1, PCB1.P$19
- new net SPI_SCLK: JP5.5, PCB1.P$23
- new net TX: JP6.6, PCB1.P$8
- net +3V3: now also C9.2, JP6.4, SJ1.2, SJ2.2, SJ3.2, SJ4.2, U5.12
- net +5V: now also C12.1, D1.A, JP6.2, L1.P$1; no longer C2.2, C6.2, C8.2, U1.1, U3.1, U4.1
- net GND: now also C10.1, C11.2, C12.2, C16.2, C9.1, IC1.GND, J1.1, JP5.6, JP6.1, U5.6, U5.PAD
- net N$1: now also JP1.4; no longer JP1.1
- net N$10: now also JP3.4; no longer JP3.1
- net N$11: now also JP3.3; no longer JP3.2
- net N$12: now also JP3.2; no longer JP3.3
- net N$13: now also JP3.1; no longer JP3.4
- net N$2: now also JP1.3; no longer JP1.2
- net N$3: now also JP1.2; no longer JP1.3
- net N$5: now also JP1.1; no longer JP1.4
- net N$6: now also JP2.4; no longer JP2.1
- net N$7: now also JP2.3; no longer JP2.2
- net N$8: now also JP2.2; no longer JP2.3
- net N$9: now also JP2.1; no longer JP2.4
Routing:
- net +12V: track 0.00 -> 98.9 mm, vias 0 -> 4
- net MD4_A2: track 0.00 -> 67.8 mm, vias 0 -> 2
- net +5V: track 150.3 -> 93.9 mm, vias 3 -> 0
- net TX: track 0.00 -> 53.3 mm, vias 0 -> 2
- net MD3_MODE: track 52.8 -> 0.00 mm
- net MD1_MODE: track 51.9 -> 0.00 mm
- net GPIO4: track 0.00 -> 51.0 mm, vias 0 -> 2
- net MD2_MODE: track 50.6 -> 0.00 mm, vias 1 -> 0
- net RX: track 0.00 -> 49.7 mm, vias 0 -> 2
- net MD4_B1: track 0.00 -> 46.3 mm
- net MD4_B2: track 0.00 -> 43.4 mm
- net MD4_A1: track 0.00 -> 42.2 mm, vias 0 -> 2
- net +3V3: track 107.0 -> 130.0 mm, vias 6 -> 9
- net SPI_SCLK: track 0.00 -> 21.1 mm
- net SPI_MOSI: track 0.00 -> 20.5 mm, vias 0 -> 2
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Other:
- outline, holes or cut-outs redrawn
- board text added: "Nekoraja Board"
- board text added: "Picam360"
- board text added: "Rev.0.2"
