File: nekojara/nekojara_board/nekojara_board.sch (EAGLE design)
At the start: 18 parts, among them U1 DRV8835, U2 MPU-9250, U3 DRV8835, U4 DRV8835

Commit message: nekojara
Parts:
- added C10, C9: 100n, resistor:C-EUC0402
- added C11, C12: 22u, resistor:C-EUC0603
- added C16: 10u, resistor:C-EUC0603
- added D1: 1N34A, diode:1N34A
- added IC1: V7805-1000, openblw:VR_1OUTXX
- added J1: (no value), con-jack:JACK-PLUG0
- added JP4: (no value), pinhead:PINHD-1X4M
- added JP5, JP6: (no value), pinhead+:PINHD-2X3
- added L1: SRN4018-100M(10u), openblw:BOURNS-SRN4018
- added SJ1, SJ2, SJ3, SJ4: SOLDERJUMPERNO, SparkFun-Retired:SOLDERJUMPERNO
- added U5: DRV8835, bt_motordriver:DRV8835
- JP1, JP2, JP3: device pinhead:PINHD-1X4 -> pinhead:PINHD-1X4M
- PCB1: device e14_Rpi3_RevA:RPI3 -> nekojara_board:RPI3
Connections:
- removed net MD1_MODE: PCB1.GPIO27, U1.MODE
- removed net MD2_MODE: PCB1.GPIO16, U3.MODE
- removed net MD3_MODE: PCB1.GPIO19, U4.MODE
- new net +12V: C10.2, C16.1, C2.2, C6.2, C8.2, D1.C, IC1.IN, J1.3, U1.VM, U3.VM, U4.VM, U5.VM
- new net GPIO4: JP6.3, PCB1.GPIO4
- new net MD4_A1: PCB1.GPIO26, U5.AIN1/APHASE
- new net MD4_A2: PCB1.GPIO27, U5.AIN2/AENBL
- new net MD4_B1: PCB1.GPIO16, U5.BIN1/BPHASE
- new net MD4_B2: PCB1.GPIO19, U5.BIN2/BENBL
- new net N$14: JP4.3, U5.AOUT2
- new net N$15: JP4.2, U5.BOUT1
- new net N$16: JP4.1, U5.BOUT2
- new net N$17: SJ4.1, U5.MODE
- new net N$18: SJ3.1, U4.MODE
- new net N$19: SJ2.1, U3.MODE
- new net N$20: SJ1.1, U1.MODE
- new net N$22: C11.1, IC1.OUT, L1.2
- new net N$4: JP4.4, U5.AOUT1
- new net RX: JP6.5, PCB1.GPIO15
- new net SPI_CE0_N: JP5.2, PCB1.GPIO8
- new net SPI_CE1_N: JP5.4, PCB1.GPIO7
- new net SPI_MISO: JP5.3, PCB1.GPIO9
- new net SPI_MOSI: JP5.1, PCB1.GPIO10
- new net SPI_SCLK: JP5.5, PCB1.GPIO11
- new net TX: JP6.6, PCB1.GPIO14
- net +3V3: now also C9.2, JP6.4, SJ1.2, SJ2.2, SJ3.2, SJ4.2, U5.VCC
- net +5V: now also C12.1, D1.A, JP6.2, L1.1; no longer C2.2, C6.2, C8.2, U1.VM, U3.VM, U4.VM
- net GND: now also C10.1, C11.2, C12.2, C16.2, C9.1, IC1.GND, J1.1, JP5.6, JP6.1, U5.GND1, U5.GND2
- net N$1: now also JP1.4; no longer JP1.1
- net N$10: now also JP3.4; no longer JP3.1
- net N$11: now also JP3.3; no longer JP3.2
- net N$12: now also JP3.2; no longer JP3.3
- net N$13: now also JP3.1; no longer JP3.4
- net N$2: now also JP1.3; no longer JP1.2
- net N$3: now also JP1.2; no longer JP1.3
- net N$5: now also JP1.1; no longer JP1.4
- net N$6: now also JP2.4; no longer JP2.1
- net N$7: now also JP2.3; no longer JP2.2
- net N$8: now also JP2.2; no longer JP2.3
- net N$9: now also JP2.1; no longer JP2.4
Other:
- moved on the sheet: C1, C2, C5, C6, C7, C8, JP1, JP2, JP3, U1, U3, U4
