File: nekojara/slipring/slipringsch.brd (EAGLE design)
At the start: 52.5 x 49 mm, 2 parts

Commit message: nekojara
Parts:
- removed JP2, JP3: (no value), pinhead+:1X01
- added JP1: (no value), pinhead:1X02M
Connections:
- net N1: now also JP1.2; no longer JP3.1
- net P1: now also JP1.1; no longer JP2.1
Routing:
- net P1: track 121.5 -> 120.6 mm
- net N1: track 142.3 -> 141.7 mm
Other:
- board text added: "nekojara360 slipring v.0.2"
