File: nekojara/slipring/slipringsch.sch (EAGLE design)
At the start: 2 parts

Commit message: nekojara
Parts:
- removed JP2, JP3: (no value), pinhead+:PINHD-1X1
- added JP1: (no value), pinhead:PINHD-1X2M
Connections:
- net N1: now also JP1.2; no longer JP3.1
- net P1: now also JP1.1; no longer JP2.1
Changed lines of the file:
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@@
 <layers>
 <layer number="1" name="Top" color="4" fill="1" visible="no" active="no"/>
+<layer number="2" name="Route2" color="1" fill="3" visible="no" active="no"/>
+<layer number="15" name="Route15" color="4" fill="6" visible="no" active="no"/>
 <layer number="16" name="Bottom" color="1" fill="1" visible="no" active="no"/>
 <layer number="17" name="Pads" color="2" fill="1" visible="no" active="no"/>
@@
 </classes>
 <parts>
-<part name="JP2" library="pinhead+" deviceset="PINHD-1X1" device=""/>
-<part name="JP3" library="pinhead+" deviceset="PINHD-1X1" device=""/>
+<part name="JP1" library="pinhead" deviceset="PINHD-1X2" device="M"/>
 </parts>
 <sheets>
@@
 </plain>
 <instances>
-<instance part="JP2" gate="G$1" x="38.1" y="43.18"/>
-<instance part="JP3" gate="G$1" x="38.1" y="35.56"/>
+<instance part="JP1" gate="G$1" x="38.1" y="38.1"/>
 </instances>
 <busses>
@@
 <segment>
 <label x="7.62" y="45.72" size="1.778" layer="95" rot="R90" xref="yes"/>
-<pinref part="JP2" gate="G$1" pin="1"/>
 <wire x1="7.62" y1="43.18" x2="7.62" y2="45.72" width="0.1524" layer="91"/>
-<wire x1="35.56" y1="43.18" x2="7.62" y2="43.18" width="0.1524" layer="91"/>
+<wire x1="25.4" y1="43.18" x2="7.62" y2="43.18" width="0.1524" layer="91"/>
+<wire x1="25.4" y1="43.18" x2="25.4" y2="40.64" width="0.1524" layer="91"/>
+<pinref part="JP1" gate="G$1" pin="1"/>
+<wire x1="25.4" y1="40.64" x2="35.56" y2="40.64" width="0.1524" layer="91"/>
 </segment>
 </net>
@@
 <segment>
 <label x="7.62" y="27.94" size="1.778" layer="95" rot="R270" xref="yes"/>
-<pinref part="JP3" gate="G$1" pin="1"/>
 <wire x1="7.62" y1="35.56" x2="7.62" y2="27.94" width="0.1524" layer="91"/>
-<wire x1="7.62" y1="35.56" x2="35.56" y2="35.56" width="0.1524" layer="91"/>
+<wire x1="7.62" y1="35.56" x2="20.32" y2="35.56" width="0.1524" layer="91"/>
+<pinref part="JP1" gate="G$1" pin="2"/>
+<wire x1="20.32" y1="35.56" x2="20.32" y2="38.1" width="0.1524" layer="91"/>
+<wire x1="20.32" y1="38.1" x2="35.56" y2="38.1" width="0.1524" layer="91"/>
 </segment>
 </net>
