File: ugv/slipring/slipringsch.brd (EAGLE design)
At the start: 52.5 x 49 mm, 1 part

Commit message: ugv : before v1.0
Routing:
- net P1: track 120.6 -> 117.9 mm
- net N1: track 141.7 -> 144.3 mm
Other:
- board text added: "Picam360 slipring v.0.3"
- board text removed: "nekojara360 slipring v.0.2"
