File: ugv/ugv_board/ugv_board.sch (EAGLE design)
At the start: 35 parts, among them IC1 V7805-1000, U1 DRV8835, U2 MPU-9250, U3 DRV8835, U4 DRV8835, U5 DRV8835

Commit message: ugv : before v1.0
Parts:
- PCB1: device nekojara_board:RPI3 -> ugv_board:RPI3
- SJ1, SJ2, SJ3, SJ4: value SOLDERJUMPERNO -> SOLDERJUMPERNC; device SparkFun-Retired:SOLDERJUMPERNO -> SparkFun-Retired:SOLDERJUMPERNC
Connections:
- net MD3_A2: now also PCB1.GPIO12; no longer PCB1.GPIO6
- net MD3_B1: now also PCB1.GPIO6; no longer PCB1.GPIO12
Other:
- note added: "Raspberry Pi extension board 4 Motor Driver"
- note added: "Rev0.3"
