File: ugv/usb/usb.brd (EAGLE design)
At the start: 13 x 12 mm, 5 parts, among them X1 USBPCB

Commit message: ugv : before v1.0
Parts:
- removed JP1, JP2, JP3, JP4: (no value), pinhead+:1X01
- added JP5: (no value), pinhead:1X04M
Connections:
- net 5V: now also JP5.1; no longer JP3.1
- net GND: now also JP5.4; no longer JP4.1
- net USB_N: now also JP5.2; no longer JP2.1
- net USB_P: now also JP5.3; no longer JP1.1
Changed lines of the file:
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@@
 </autorouter>
 <elements>
-<element name="JP2" library="pinhead+" package="1X01" value="" x="10.922" y="4.699" smashed="yes">
-<attribute name="VALUE" x="9.652" y="1.524" size="1.27" layer="27"/>
-</element>
-<element name="JP3" library="pinhead+" package="1X01" value="" x="10.922" y="2.159" smashed="yes">
-<attribute name="VALUE" x="9.652" y="-1.016" size="1.27" layer="27"/>
-</element>
 <element name="X1" library="usb" package="USB-A-PCB" value="USBPCB" x="5" y="6"/>
-<element name="JP1" library="pinhead+" package="1X01" value="" x="10.922" y="7.239" smashed="yes">
-<attribute name="VALUE" x="9.652" y="4.064" size="1.27" layer="27"/>
-</element>
-<element name="JP4" library="pinhead+" package="1X01" value="" x="10.922" y="9.779" smashed="yes">
-<attribute name="VALUE" x="9.652" y="6.604" size="1.27" layer="27"/>
-</element>
+<element name="JP5" library="pinhead" package="1X04M" value="" x="10.922" y="5.969" rot="R90"/>
 </elements>
 <signals>
 <signal name="USB_P">
 <contactref element="X1" pad="USB_P"/>
-<contactref element="JP1" pad="1"/>
-<wire x1="10.922" y1="7.239" x2="10.683" y2="7" width="1.016" layer="1"/>
-<wire x1="10.683" y1="7" x2="5.3" y2="7" width="1.016" layer="1"/>
+<contactref element="JP5" pad="3"/>
+<wire x1="5.3" y1="7" x2="10.891" y2="7" width="0.1524" layer="1"/>
+<wire x1="10.891" y1="7" x2="10.922" y2="6.969" width="0.1524" layer="1"/>
 </signal>
 <signal name="USB_N">
 <contactref element="X1" pad="USB_M"/>
-<contactref element="JP2" pad="1"/>
-<wire x1="10.922" y1="4.699" x2="10.621" y2="5" width="1.016" layer="1"/>
-<wire x1="10.621" y1="5" x2="5.3" y2="5" width="1.016" layer="1"/>
+<contactref element="JP5" pad="2"/>
+<wire x1="5.3" y1="5" x2="10.891" y2="5" width="0.2" layer="1"/>
+<wire x1="10.891" y1="5" x2="10.922" y2="4.969" width="0.2" layer="1"/>
 </signal>
 <signal name="5V">
 <contactref element="X1" pad="5V"/>
-<contactref element="JP3" pad="1"/>
-<wire x1="10.922" y1="2.159" x2="10.581" y2="2.5" width="1.016" layer="1"/>
-<wire x1="10.581" y1="2.5" x2="4.8" y2="2.5" width="1.016" layer="1"/>
+<contactref element="JP5" pad="1"/>
+<wire x1="4.8" y1="2.5" x2="10.453" y2="2.5" width="1.27" layer="1"/>
+<wire x1="10.453" y1="2.5" x2="10.922" y2="2.969" width="1.27" layer="1"/>
 </signal>
 <signal name="GND">
 <contactref element="X1" pad="GND"/>
-<contactref element="JP4" pad="1"/>
 <polygon width="0.2" layer="16">
 <vertex x="0" y="0"/>
@@
 <vertex x="0" y="12"/>
 </polygon>
-<wire x1="10.922" y1="9.779" x2="10.643" y2="9.5" width="0.8128" layer="1"/>
-<wire x1="10.643" y1="9.5" x2="4.8" y2="9.5" width="0.8128" layer="1"/>
+<contactref element="JP5" pad="4"/>
+<wire x1="4.8" y1="9.5" x2="10.391" y2="9.5" width="1.27" layer="1"/>
+<wire x1="10.391" y1="9.5" x2="10.922" y2="8.969" width="1.27" layer="1"/>
 </signal>
 </signals>
