File: ugv/usb/usb.sch (EAGLE design)
At the start: 5 parts, among them X1 USBPCB

Commit message: ugv : before v1.0
Parts:
- removed JP1, JP2, JP3, JP4: (no value), pinhead+:PINHD-1X1
- added JP5: (no value), pinhead:PINHD-1X4M
Connections:
- net 5V: now also JP5.1; no longer JP3.1
- net GND: now also JP5.4; no longer JP4.1
- net USB_N: now also JP5.2; no longer JP2.1
- net USB_P: now also JP5.3; no longer JP1.1
Changed lines of the file:
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@@
 </classes>
 <parts>
-<part name="JP2" library="pinhead+" deviceset="PINHD-1X1" device=""/>
-<part name="JP3" library="pinhead+" deviceset="PINHD-1X1" device=""/>
 <part name="X1" library="usb" deviceset="USB" device="PCB"/>
-<part name="JP1" library="pinhead+" deviceset="PINHD-1X1" device=""/>
-<part name="JP4" library="pinhead+" deviceset="PINHD-1X1" device=""/>
+<part name="JP5" library="pinhead" deviceset="PINHD-1X4" device="M"/>
 </parts>
 <sheets>
@@
 </plain>
 <instances>
-<instance part="JP2" gate="G$1" x="22.86" y="43.18"/>
-<instance part="JP3" gate="G$1" x="22.86" y="35.56"/>
 <instance part="X1" gate="G$1" x="45.72" y="35.56"/>
-<instance part="JP1" gate="G$1" x="22.86" y="50.8"/>
-<instance part="JP4" gate="G$1" x="22.86" y="27.94"/>
+<instance part="JP5" gate="A" x="20.32" y="38.1" rot="MR0"/>
 </instances>
 <busses>
@@
 <wire x1="43.18" y1="43.18" x2="35.56" y2="43.18" width="0.1524" layer="91"/>
 <wire x1="35.56" y1="43.18" x2="35.56" y2="50.8" width="0.1524" layer="91"/>
-<pinref part="JP1" gate="G$1" pin="1"/>
-<wire x1="35.56" y1="50.8" x2="20.32" y2="50.8" width="0.1524" layer="91"/>
+<wire x1="35.56" y1="50.8" x2="15.24" y2="50.8" width="0.1524" layer="91"/>
+<wire x1="15.24" y1="50.8" x2="15.24" y2="38.1" width="0.1524" layer="91"/>
+<pinref part="JP5" gate="A" pin="3"/>
+<wire x1="15.24" y1="38.1" x2="22.86" y2="38.1" width="0.1524" layer="91"/>
 </segment>
 </net>
@@
 <segment>
 <pinref part="X1" gate="G$1" pin="D-"/>
-<wire x1="43.18" y1="40.64" x2="30.48" y2="40.64" width="0.1524" layer="91"/>
-<wire x1="30.48" y1="40.64" x2="30.48" y2="43.18" width="0.1524" layer="91"/>
-<pinref part="JP2" gate="G$1" pin="1"/>
-<wire x1="30.48" y1="43.18" x2="20.32" y2="43.18" width="0.1524" layer="91"/>
+<wire x1="43.18" y1="40.64" x2="22.86" y2="40.64" width="0.1524" layer="91"/>
+<pinref part="JP5" gate="A" pin="2"/>
 </segment>
 </net>
@@
 <pinref part="X1" gate="G$1" pin="VBUS"/>
 <wire x1="43.18" y1="38.1" x2="30.48" y2="38.1" width="0.1524" layer="91"/>
-<wire x1="30.48" y1="38.1" x2="30.48" y2="35.56" width="0.1524" layer="91"/>
-<pinref part="JP3" gate="G$1" pin="1"/>
-<wire x1="30.48" y1="35.56" x2="20.32" y2="35.56" width="0.1524" layer="91"/>
+<wire x1="30.48" y1="38.1" x2="30.48" y2="43.18" width="0.1524" layer="91"/>
+<pinref part="JP5" gate="A" pin="1"/>
+<wire x1="30.48" y1="43.18" x2="22.86" y2="43.18" width="0.1524" layer="91"/>
 </segment>
 </net>
@@
 <wire x1="43.18" y1="35.56" x2="35.56" y2="35.56" width="0.1524" layer="91"/>
 <wire x1="35.56" y1="35.56" x2="35.56" y2="27.94" width="0.1524" layer="91"/>
-<pinref part="JP4" gate="G$1" pin="1"/>
-<wire x1="35.56" y1="27.94" x2="20.32" y2="27.94" width="0.1524" layer="91"/>
+<wire x1="35.56" y1="27.94" x2="15.24" y2="27.94" width="0.1524" layer="91"/>
+<wire x1="15.24" y1="27.94" x2="15.24" y2="35.56" width="0.1524" layer="91"/>
+<pinref part="JP5" gate="A" pin="4"/>
+<wire x1="15.24" y1="35.56" x2="22.86" y2="35.56" width="0.1524" layer="91"/>
 </segment>
 </net>
