File: usv/usv_50w_board/usv_50w_board.brd (EAGLE design)
At the start: 65 x 30 mm, 27 parts, among them IC1 ADS7828E/250G4, J1 B4B-PH-K-S(LF)(SN), J2 10118193-0001LF, J3 B4B-PH-K-S(LF)(SN), J4 B4B-PH-K-S(LF)(SN), J5 B4B-PH-K-S(LF)(SN), Q1 IRLML6346TRPBF, U2 MPU-9250

Commit message: usv50w
Parts:
- moved U2 0.20 mm to (41.3, 16.3)
Connections:
- net USB_5V renamed USB_D_N
- net USB_D- renamed USB_D_P
Routing:
- net PWM1: track 27.5 -> 33.4 mm, vias 0 -> 1
- net +5V: track 104.9 -> 99.6 mm
- net PWM2: track 27.3 -> 31.9 mm, vias 0 -> 1
- net USB_D_N: track 12.3 -> 16.1 mm, vias 0 -> 1
- net PWM3: track 32.2 -> 35.7 mm, vias 0 -> 1
- net +3V3: track 81.2 -> 83.5 mm
- net PWM4: track 28.6 -> 30.6 mm, vias 0 -> 1
- net GPS_TX: track 21.5 -> 23.3 mm, vias 0 -> 1
- net GPS_RX: track 31.0 -> 32.5 mm, vias 0 -> 1
- net USB_D_P: track 15.9 -> 17.4 mm, vias 0 -> 1
- net AGND: vias 12 -> 19
- removed copper zone on layer 2, net AGND
- removed copper zone on layer 2, net GND
