File: usv/usv_50w_board/usv_50w_board.sch (EAGLE design)
At the start: 26 parts, among them IC1 ADS7828E/250G4, J1 B4B-PH-K-S(LF)(SN), J2 10118193-0001LF, J3 B4B-PH-K-S(LF)(SN), J4 B4B-PH-K-S(LF)(SN), J5 B4B-PH-K-S(LF)(SN), Q1 IRLML6346TRPBF, U2 MPU-9250

Commit message: usv50w
Connections:
- net USB_5V renamed USB_D_N
- net USB_D- renamed USB_D_P
Changed lines of the file:
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@@
 </segment>
 </net>
-<net name="USB_5V" class="0">
+<net name="USB_D_N" class="3">
 <segment>
 <pinref part="J2" gate="G$1" pin="D-"/>
@@
 </segment>
 </net>
-<net name="USB_D-" class="0">
+<net name="USB_D_P" class="3">
 <segment>
 <pinref part="J2" gate="G$1" pin="D+"/>

Commit message: usv 50w rev0.2
Parts:
- added C8: 10u, resistor:C-USC0603
- added Q2: P-CHANNEL-MOSFET, GeekAmmo:P-CHANNEL-MOSFET
- added R10, R12, R13, R15, R17: 100k, resistor:R-US_R0603
- added R11: 500k, resistor:R-US_R0603
- added R14, R16, R18, R19, R20, R9: 10k, resistor:R-US_R0603
- added SJ1: SOLDERJUMPERTRACE, SparkFun-Retired:SOLDERJUMPERTRACE
- added U1: V7812W-500R, V7812W-500R:V7812W-500R
- C5, C6, C7: value 4.7u -> 10u
- JP1: device pinhead:PINHD-1X3 -> pinhead+:PINHD-1X4
- Q1: value IRLML6346TRPBF -> P-CHANNEL-MOSFET; device openblw:NMOS-FETSOT23 -> GeekAmmo:P-CHANNEL-MOSFET
- R5: value 100k -> 500k
- R8: value 100k -> 10k
Connections:
- net 12VBAT_SENSE renamed SOLAR_SENSE
- net 12VBAT_SRC renamed SOLAR_V
- removed net RX1_SENSE: C5.2, IC1.CH1, R4.1
- removed net RX1_SRC: J3.2, R4.2
- removed net RX2_SENSE: C6.2, IC1.CH2, R5.1
- removed net RX2_SRC: J3.3, R5.2
- removed net RX3_SENSE: C7.2, IC1.CH3, R8.1
- removed net RX3_SRC: J3.4, R8.2
- new net 12V: J3.3, R5.2, U1.VIN_P
- new net 12V_SENSE: IC1.CH2, R10.1, R5.1
- new net BAT_SENSE: IC1.CH1, R11.1, R12.1
- new net BAT_V: J3.2, R11.2
- new net EXT1_V: J4.1, R4.2
- new net EXT2_V: J4.2, R13.2
- new net EXT3_V: J4.3, R15.2
- new net EXT4_V: J4.4, R17.2
- new net GPS_1PPS: JP2.5, R8.2
- new net GPS_5V: JP2.1, Q2.D
- new net GPS_ENABLE: Q2.G, R20.2, U$3.GPIO5
- new net N$2: R8.1, U$3.GPIO22/GEN3
- new net N$3: R14.1, U$3.GPIO27/GEN2
- new net N$5: R16.1, U$3.GPIO17/GEN0
- new net N$7: R19.2, U$3.GPIO18
- new net RESERVED: IC1.CH3
- new net USB_5V: J1.1, Q1.D
- net +3V3: now also JP1.1
- net +5V: now also Q1.S, Q2.S, R20.1, R9.1, U1.VO_P; no longer J1.1, J2.VUSB, JP1.1, JP2.1
- net AGND: now also C5.2, C6.2, C7.2, C8.2, JP1.4, R10.2, R12.2, SJ1.1; no longer C5.1, C6.1, C7.1, JP1.3
- net EXT1_SENSE: now also C5.1, R4.1; no longer J4.1
- net EXT2_SENSE: now also C6.1, R13.1; no longer J4.2
- net EXT3_SENSE: now also C7.1, R15.1; no longer J4.3
- net EXT4_SENSE: now also C8.1, R17.1; no longer J4.4
- net GND: now also J1.4, J3.4, SJ1.2, U1.GND; no longer JP1.2, Q1.S
- net N$6: now also R18.2, U$3.GEN5/GPIO24; no longer J1.4, Q1.D
- net PWM1: now also R14.2; no longer U$3.GPIO17/GEN0
- net PWM2: now also R16.2; no longer U$3.GPIO27/GEN2
- net PWM3: now also R18.1; no longer U$3.GPIO18
- net PWM4: now also R19.1; no longer U$3.GEN4/GPIO23
- net TWI_SCL: now also JP1.3
- net TWI_SDA: now also JP1.2
- net USB_ENABLE: now also R9.2, U$3.GPIO6; no longer U$3.GPIO5
Other:
- note added: "DCDC"
- moved on the sheet: C5, C6, C7, J1, J2, J5, JP2, R2, R3, R4, R5, R8

Commit message: usv 50w 0.3
Parts:
- removed Q1, Q2: P-CHANNEL-MOSFET, GeekAmmo:P-CHANNEL-MOSFET
- removed R20, R8, R9: 10k, resistor:R-US_R0603
- added C10, C11, C13: 10u, resistor:C-USC0603
- added C12, C14, C9: 100n, resistor:C-USC0603
- added U$1: AP2166S, diodes-inc:AP2166S
- JP1: device pinhead+:PINHD-1X4 -> pinhead+:PINHD-1X5
Connections:
- removed net N$2: R8.1, U$3.GPIO22/GEN3
- removed net RESERVED: IC1.CH3
- removed net USB_D_N: J1.2, J2.D-
- removed net USB_D_P: J1.3, J2.D+
- new net D_N: J1.3, J2.D-
- new net D_P: J1.2, J2.D+
- net +3V3: now also JP1.2; no longer JP1.1, U$3.3V3@2
- net +5V: now also C10.1, C14.1, U$1.IN; no longer Q1.S, Q2.S, R20.1, R9.1
- net AGND: no longer JP1.4
- net GND: now also C10.2, C11.2, C12.2, C13.2, C14.2, C9.2, IC1.CH3, J1.1, JP1.5, U$1.GND; no longer J1.4
- net GPS_1PPS: now also U$3.GPIO22/GEN3; no longer R8.2
- net GPS_5V: now also C12.1, C13.1, JP1.1, U$1.OUTB; no longer Q2.D
- net GPS_ENABLE: now also U$1.!ENB!; no longer Q2.G, R20.2
- net TWI_SCL: now also JP1.4; no longer JP1.3
- net TWI_SDA: now also JP1.3; no longer JP1.2
- net USB_5V: now also C11.1, C9.1, J1.4, U$1.OUTA; no longer J1.1, Q1.D
- net USB_ENABLE: now also U$1.!ENA!; no longer Q1.G, R9.2
Other:
- moved on the sheet: J1
