File: usv/trickle_charger/trickle_charger.brd (EAGLE design)
At the start: 65 x 30 mm, 23 parts, among them IC1 LM358, J1 B4B-PH-K-S(LF)(SN), J2 B4B-PH-K-S(LF)(SN), J3 B4B-PH-K-S(LF)(SN), J4 B4B-PH-K-S(LF)(SN), Q1 IRLML6346TRPBF

Commit message: usv 50w 0.3
Parts:
- removed JP10, JP4, JP5, JP6, JP7, JP8, JP9: (no value), pinhead+:1X02
- added H1, H10, H11, H12, H13, H14, H2, H3, H4, H5, H6, H7, H8, H9: SEW_HOLE-SMALL, LilyPad-Wearables:SIMPLE_HOLE_SM
- added R7: 200, resistor:R0603
- added R8: 10k, resistor:R0603
- R4: value 470 -> 200
- moved LOGO1 15.5 mm to (60.9, 13.8)
- moved Q1 1.27 mm to (6.35, 14.6)
- moved R4 1.27 mm to (6.35, 19.1)
- moved R5 0.90 mm to (36.2, 13.3)
- moved R6 0.64 mm to (23.5, 13.3)
Connections:
- removed net SW_BAT-: IC1.4, JP6.2, JP9.2, Q1.2
- removed net USB_ENABLE: IC1.1, Q1.1
- removed net V-: D1.P$2, D2.A, JP4.2, JP8.2, R3.1
- new net N$5: IC1.1, R7.2
- new net N$6: Q1.1, R7.1, R8.1
- new net SOLAR+: R6.1
- new net SOLAR-: H10.P$1, H2.P$1, IC1.4, Q1.2, R8.2
- new net SW_BAT+: H12.P$1, H6.P$1
- net BAT+: now also H3.P$1; no longer JP5.1
- net BAT-: now also D1.P$2, D2.A, H4.P$1, H5.P$1, R3.1; no longer JP5.2, JP6.1
- net N$1: now also IC1.3; no longer IC1.2
- net N$13: now also H9.P$1; no longer JP8.1
- net N$14: now also H11.P$1; no longer JP9.1
- net N$3: now also IC1.2; no longer IC1.3
- net OUT+: now also H13.P$1, H7.P$1; no longer JP10.1, JP7.1
- net OUT-: now also H14.P$1, H8.P$1; no longer JP10.2, JP7.2
- net V+: now also H1.P$1; no longer JP4.1, R6.1
Routing:
- net BAT-: track 0.00 -> 54.3 mm
- net SW_BAT-: track 52.0 -> 0.00 mm
- net SOLAR-: track 0.00 -> 45.1 mm
- net V-: track 28.5 -> 0.00 mm
- net USB_ENABLE: track 18.4 -> 0.00 mm
- net N$5: track 0.00 -> 17.2 mm, vias 0 -> 1
- net N$6: track 0.00 -> 7.09 mm
- net V+: track 36.8 -> 30.0 mm
- net OUT-: track 26.7 -> 33.4 mm
- net OUT+: track 25.8 -> 29.7 mm
- net N$3: track 15.8 -> 12.5 mm
- net N$2: track 9.54 -> 8.27 mm
- net N$1: track 19.9 -> 18.8 mm
- net BAT+: track 13.1 -> 12.2 mm
- added copper zone on layer 1, net BAT-
- added copper zone on layer 1, net SOLAR-
- added copper zone on layer 1, net SW_BAT+
- removed copper zone on layer 16, net BAT-
- removed copper zone on layer 1, net SW_BAT-
- removed copper zone on layer 1, net V-
Other:
- board text added: "BAT+"
- board text added: "BAT-"
- board text added: "OUT+"
- board text added: "OUT-"
- board text added: "Rev.0.2"
- board text added: "SOLAR+"
- board text added: "SOLAR-"
- board text added: "SW_BAT+"
- board text added: "SW_BAT-"
- board text removed: "Rev.0.1"
