File: usv/trickle_charger/trickle_charger.sch (EAGLE design)
At the start: 22 parts, among them IC1 LM358, J1 B4B-PH-K-S(LF)(SN), J2 B4B-PH-K-S(LF)(SN), J3 B4B-PH-K-S(LF)(SN), J4 B4B-PH-K-S(LF)(SN), Q1 IRLML6346TRPBF

Commit message: usv 50w 0.3
Parts:
- removed JP10, JP4, JP5, JP6, JP7, JP8, JP9: (no value), pinhead+:PINHD-1X2
- added H1, H10, H11, H12, H13, H14, H2, H3, H4, H5, H6, H7, H8, H9: SEW_HOLE-SMALL, LilyPad-Wearables:SEW_HOLE-SMALL
- added R7: 200, resistor:R-US_R0603
- added R8: 10k, resistor:R-US_R0603
- R4: value 470 -> 200
Connections:
- removed net SW_BAT-: IC1G1.V-, JP6.2, JP9.2, Q1.S
- removed net USB_ENABLE: IC1G1.OUT, Q1.G
- removed net V-: D1.A, D2.A, JP4.2, JP8.2, R3.1
- new net N$5: IC1G1.OUT, R7.2
- new net N$6: Q1.G, R7.1, R8.1
- new net SOLAR+: R6.1
- new net SOLAR-: H10.P$1, H2.P$1, IC1G1.V-, Q1.S, R8.2
- new net SW_BAT+: H12.P$1, H6.P$1
- net BAT+: now also H3.P$1; no longer JP5.1
- net BAT-: now also D1.A, D2.A, H4.P$1, H5.P$1, R3.1; no longer JP5.2, JP6.1
- net N$1: now also IC1G1.+IN; no longer IC1G1.-IN
- net N$13: now also H9.P$1; no longer JP8.1
- net N$14: now also H11.P$1; no longer JP9.1
- net N$3: now also IC1G1.-IN; no longer IC1G1.+IN
- net OUT+: now also H13.P$1, H7.P$1; no longer JP10.1, JP7.1
- net OUT-: now also H14.P$1, H8.P$1; no longer JP10.2, JP7.2
- net V+: now also H1.P$1; no longer JP4.1, R6.1
Other:
- moved on the sheet: D2, Q1, R4
