File: usv/usv_board/usv_board.brd (EAGLE design)
At the start: 53.3 x 59.7 mm, 15 parts, among them IC1 74157N, J1 ARDUINO_R3_SHIELD, Q1 PFETBS250

Commit message: usv 50w 0.3
Parts:
- removed JP6: (no value), pinhead+:1X02
- removed Q1: PFETBS250, adafruit:TO92-OVAL
- removed R3: 10k, resistor:0207/7
- added C1: 4.7u, resistor:E2-4
- R2: value 10k -> 100k
- moved JP5 17.8 mm to (10.3, 34.2), turned to 270 degrees
- moved R2 11.8 mm to (20.3, 36.8), turned to 180 degrees
- moved JP4 10.2 mm to (10.3, 42.5)
- moved JP3 8.89 mm to (10.3, 50.8)
- moved JP2 1.27 mm to (11.6, 12.7)
Connections:
- removed net MASTER_RX: J1.TX, JP5.2
- removed net MASTER_TX: J1.RX, JP5.4
- removed net V_AUX: JP5.1, Q1.3, R2.2
- removed net V_WAKEUP: JP5.3, Q1.1, R3.2
- removed net WAKEUP: J1.D8, Q1.2, R2.1
- new net AUTO_LP: C1.+, J1.A3, JP5.2, R2.1
- new net AUTO_PROPO: JP5.1, R2.2
- net +5V: now also JP3.3, JP3.4, JP4.3, JP4.4, JP5.3, JP5.4; no longer JP3.1, JP3.2, JP4.1, JP4.2
- net AUTO_MODE: no longer JP6.1
- net GND: now also C1.-; no longer JP6.2, R3.1
- net RUDDER_OUTPUT: now also JP3.2; no longer JP3.4
- net RUDDER_PROPO: now also JP3.1; no longer J1.D3, JP3.3
- net SKREW_OUTPUT: now also JP4.2; no longer JP4.4
- net SKREW_PROPO: now also JP4.1; no longer JP4.3
Routing:
- net AUTO_LP: track 0.00 -> 65.1 mm, vias 0 -> 2
- net WAKEUP: track 34.8 -> 0.00 mm
- net V_WAKEUP: track 15.8 -> 0.00 mm
- net V_AUX: track 13.8 -> 0.00 mm
- net +5V: track 117.0 -> 128.2 mm
- net AUTO_PROPO: track 0.00 -> 8.53 mm
- net RUDDER_PROPO: track 39.5 -> 31.8 mm
- net MASTER_RX: track 7.52 -> 0.00 mm
- net MASTER_TX: track 7.52 -> 0.00 mm
- net AUTO_MODE: track 62.7 -> 68.4 mm
- net SKREW_PWM: track 40.3 -> 36.2 mm
- net RUDDER_OUTPUT: track 25.6 -> 29.3 mm
- net RUDDER_PWM: track 40.0 -> 42.5 mm
- net GPS_RX: track 32.8 -> 34.2 mm
- net GPS_TX: track 29.5 -> 28.4 mm
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Other:
- board text added: "Rev.0.2"
- board text removed: "RX"
- board text removed: "Rev.0.1"
- board text removed: "TX"
