File: usv/usv_board/usv_board.sch (EAGLE design)
At the start: 14 parts, among them IC1 74157N, J1 ARDUINO_R3_SHIELD, Q1 PFETBS250

Commit message: usv 50w 0.3
Parts:
- removed JP6: (no value), pinhead+:PINHD-1X2
- removed Q1: PFETBS250, adafruit:PFETBS250
- removed R3: 10k, resistor:R-EU_0207/7
- added C1: 4.7u, resistor:CPOL-EUE2-4
- R2: value 10k -> 100k
Connections:
- removed net MASTER_RX: J1.TX, JP5.2
- removed net MASTER_TX: J1.RX, JP5.4
- removed net V_AUX: JP5.1, Q1.S, R2.2
- removed net V_WAKEUP: JP5.3, Q1.D, R3.2
- removed net WAKEUP: J1.D8, Q1.G, R2.1
- new net AUTO_LP: C1.+, J1.A3, JP5.2, R2.1
- new net AUTO_PROPO: JP5.1, R2.2
- net +5V: now also JP3.3, JP3.4, JP4.3, JP4.4, JP5.3, JP5.4; no longer JP3.1, JP3.2, JP4.1, JP4.2
- net AUTO_MODE: no longer JP6.1
- net GND: now also C1.-; no longer JP6.2, R3.1
- net RUDDER_OUTPUT: now also JP3.2; no longer JP3.4
- net RUDDER_PROPO: now also JP3.1; no longer J1.*D3, JP3.3
- net SKREW_OUTPUT: now also JP4.2; no longer JP4.4
- net SKREW_PROPO: now also JP4.1; no longer JP4.3
Other:
- note removed: "WAKEUP"
- moved on the sheet: JP5, R2
